Commit message: cugo.xacroのoriginの設定項目の順序を統一

File: models/cugo/cugo.xacro (robot description, xacro)
@@ -34,5 +34,5 @@
     <parent link="base_link"/>
     <child  link="base_body"/>
-    <origin rpy="0 0 0" xyz="0 0 0"/>
+    <origin xyz="0 0 0" rpy="0 0 0"/>
   </joint>
   <link name="base_body">
@@ -52,5 +52,5 @@
     <parent link="base_body"/>
     <child link="body_collision"/>
-    <origin rpy="0 0 0" xyz="0 0 ${body_collision_height/2+body_height/2-0.05}"/>
+    <origin xyz="0 0 ${body_collision_height/2+body_height/2-0.05}" rpy="0 0 0"/>
   </joint>
   <link name="body_collision">
@@ -73,13 +73,13 @@
   </link>
   <joint name="left_wheel_joint" type="continuous">
-    <axis rpy="0 0 0" xyz="0 0 -1"/>
+    <axis xyz="0 0 -1" rpy="0 0 0"/>
     <limit lower="-1.57" upper="1.57" effort="0.5" velocity="2.0"/>
     <parent link="base_body"/>
     <child link="left_wheel"/>
-    <origin rpy="0 1.57075 -1.57" xyz="0 ${left_wheel_y} ${center_wheel_z}"/>
+    <origin xyz="0 ${left_wheel_y} ${center_wheel_z}" rpy="0 1.57075 -1.57"/>
   </joint>
   <link name="left_wheel">
     <visual>
-      <origin rpy="0 0 0" xyz="0 0 0"/>
+      <origin xyz="0 0 0" rpy="0 0 0"/>
       <geometry>
         <cylinder length="${wheel_length}" radius="${mini_wheel_radius}"/>
@@ -98,13 +98,13 @@
   </link>
   <joint name="left_wheel_joint_center_mini_front" type="continuous">
-    <axis rpy="0 0 0" xyz="0 0 -1"/>
+    <axis xyz="0 0 -1" rpy="0 0 0"/>
     <limit lower="-1.57" upper="1.57" effort="1.0" velocity="2.0"/>
     <parent link="base_body"/>
     <child link="left_wheel_center_mini_front"/>
-    <origin rpy="0 1.57075 -1.57" xyz="${mini_wheel_radius*2} ${left_wheel_y} ${center_wheel_z}"/>
+    <origin xyz="${mini_wheel_radius*2} ${left_wheel_y} ${center_wheel_z}" rpy="0 1.57075 -1.57"/>
   </joint>
   <link name="left_wheel_center_mini_front">
     <visual>
-      <origin rpy="0 0 0" xyz="0 0 0"/>
+      <origin xyz="0 0 0" rpy="0 0 0"/>
       <geometry>
         <cylinder length="${wheel_length}" radius="${mini_wheel_radius}"/>
@@ -123,13 +123,13 @@
   </link>
   <joint name="left_wheel_joint_center_mini_back" type="continuous">
-    <axis rpy="0 0 0" xyz="0 0 -1"/>
+    <axis xyz="0 0 -1" rpy="0 0 0"/>
     <limit lower="-1.57" upper="1.57" effort="1.0" velocity="2.0"/>
     <parent link="base_body"/>
     <child link="left_wheel_center_mini_back"/>
-    <origin rpy="0 1.57075 -1.57" xyz="-${mini_wheel_radius*2} ${left_wheel_y} ${center_wheel_z}"/>
+    <origin xyz="-${mini_wheel_radius*2} ${left_wheel_y} ${center_wheel_z}" rpy="0 1.57075 -1.57"/>
   </joint>
   <link name="left_wheel_center_mini_back">
     <visual>
-      <origin rpy="0 0 0" xyz="0 0 0"/>
+      <origin xyz="0 0 0" rpy="0 0 0"/>
       <geometry>
         <cylinder length="${wheel_length}" radius="${mini_wheel_radius}"/>
@@ -148,13 +148,13 @@
   </link>
   <joint name="left_wheel_joint_big_front" type="continuous">
-    <axis rpy="0 0 0" xyz="0 0 -1"/>
+    <axis xyz="0 0 -1" rpy="0 0 0"/>
     <limit lower="-1.57" upper="1.57" effort="1.0" velocity="2.0"/>
     <parent link="base_body"/>
     <child link="left_wheel_big_front"/>
-    <origin rpy="0 1.57075 -1.57" xyz="${big_wheel_front_x} ${left_wheel_y} ${big_wheel_z}"/>
+    <origin xyz="${big_wheel_front_x} ${left_wheel_y} ${big_wheel_z}" rpy="0 1.57075 -1.57"/>
   </joint>
   <link name="left_wheel_big_front">
     <visual>
-      <origin rpy="0 0 0" xyz="0 0 0"/>
+      <origin xyz="0 0 0" rpy="0 0 0"/>
       <geometry>
         <cylinder length="${wheel_length}" radius="${wheel_radius}"/>
@@ -173,13 +173,13 @@
   </link>
   <joint name="left_wheel_joint_big_back" type="continuous">
-    <axis rpy="0 0 0" xyz="0 0 -1"/>
+    <axis xyz="0 0 -1" rpy="0 0 0"/>
     <limit lower="-1.57" upper="1.57" effort="1.0" velocity="2.0"/>
     <parent link="base_body"/>
     <child link="left_wheel_big_back"/>
-    <origin rpy="0 1.57075 -1.57" xyz="${big_wheel_back_x} ${left_wheel_y} ${big_wheel_z}"/>
+    <origin xyz="${big_wheel_back_x} ${left_wheel_y} ${big_wheel_z}" rpy="0 1.57075 -1.57"/>
   </joint>
   <link name="left_wheel_big_back">
     <visual>
-      <origin rpy="0 0 0" xyz="0 0 0"/>
+      <origin xyz="0 0 0" rpy="0 0 0"/>
       <geometry>
         <cylinder length="${wheel_length}" radius="${wheel_radius}"/>
@@ -198,13 +198,13 @@
   </link>
   <joint name="right_wheel_joint" type="continuous">
-    <axis rpy="0 0 0" xyz="0 0 -1"/>
+    <axis xyz="0 0 -1" rpy="0 0 0"/>
     <limit lower="-1.57" upper="1.57" effort="1.0" velocity="2.0"/>
     <parent link="base_body"/>
     <child link="right_wheel"/>
-    <origin rpy="0 1.57075 -1.57" xyz="0 ${right_wheel_y} ${center_wheel_z}"/>
+    <origin xyz="0 ${right_wheel_y} ${center_wheel_z}" rpy="0 1.57075 -1.57"/>
   </joint>
   <link name="right_wheel">
     <visual>
-      <origin rpy="0 0 0" xyz="0 0 0"/>
+      <origin xyz="0 0 0" rpy="0 0 0"/>
       <geometry>
         <cylinder length="${wheel_length}" radius="${mini_wheel_radius}"/>
@@ -223,13 +223,13 @@
   </link>
   <joint name="right_wheel_joint_center_mini_front" type="continuous">
-    <axis rpy="0 0 0" xyz="0 0 -1"/>
+    <axis xyz="0 0 -1" rpy="0 0 0"/>
     <limit lower="-1.57" upper="1.57" effort="1.0" velocity="2.0"/>
     <parent link="base_body"/>
     <child link="right_wheel_center_mini_front"/>
-    <origin rpy="0 1.57075 -1.57" xyz="${mini_wheel_radius*2} ${right_wheel_y} ${center_wheel_z}"/>
+    <origin xyz="${mini_wheel_radius*2} ${right_wheel_y} ${center_wheel_z}" rpy="0 1.57075 -1.57"/>
   </joint>
   <link name="right_wheel_center_mini_front">
     <visual>
-      <origin rpy="0 0 0" xyz="0 0 0"/>
+      <origin xyz="0 0 0" rpy="0 0 0"/>
       <geometry>
         <cylinder length="${wheel_length}" radius="${mini_wheel_radius}"/>
@@ -248,13 +248,13 @@
   </link>
   <joint name="right_wheel_joint_center_mini_back" type="continuous">
-    <axis rpy="0 0 0" xyz="0 0 -1"/>
+    <axis xyz="0 0 -1" rpy="0 0 0"/>
     <limit lower="-1.57" upper="1.57" effort="1.0" velocity="2.0"/>
     <parent link="base_body"/>
     <child link="right_wheel_center_mini_back"/>
-    <origin rpy="0 1.57075 -1.57" xyz="-${mini_wheel_radius*2} ${right_wheel_y} ${center_wheel_z}"/>
+    <origin xyz="-${mini_wheel_radius*2} ${right_wheel_y} ${center_wheel_z}" rpy="0 1.57075 -1.57"/>
   </joint>
   <link name="right_wheel_center_mini_back">
     <visual>
-      <origin rpy="0 0 0" xyz="0 0 0"/>
+      <origin xyz="0 0 0" rpy="0 0 0"/>
       <geometry>
         <cylinder length="${wheel_length}" radius="${mini_wheel_radius}"/>
@@ -273,13 +273,13 @@
   </link>
   <joint name="right_wheel_joint_big_front" type="continuous">
-    <axis rpy="0 0 0" xyz="0 0 -1"/>
+    <axis xyz="0 0 -1" rpy="0 0 0"/>
     <limit lower="-1.57" upper="1.57" effort="1.0" velocity="2.0"/>
     <parent link="base_body"/>
     <child link="right_wheel_big_front"/>
-    <origin rpy="0 1.57075 -1.57" xyz="${big_wheel_front_x} ${right_wheel_y} ${big_wheel_z}"/>
+    <origin xyz="${big_wheel_front_x} ${right_wheel_y} ${big_wheel_z}" rpy="0 1.57075 -1.57"/>
   </joint>
   <link name="right_wheel_big_front">
     <visual>
-      <origin rpy="0 0 0" xyz="0 0 0"/>
+      <origin xyz="0 0 0" rpy="0 0 0"/>
       <geometry>
         <cylinder length="${wheel_length}" radius="${wheel_radius}"/>
@@ -298,13 +298,13 @@
   </link>
   <joint name="right_wheel_joint_big_back" type="continuous">
-    <axis rpy="0 0 0" xyz="0 0 -1"/>
+    <axis xyz="0 0 -1" rpy="0 0 0"/>
     <limit lower="-1.57" upper="1.57" effort="1.0" velocity="2.0"/>
     <parent link="base_body"/>
     <child link="right_wheel_big_back"/>
-    <origin rpy="0 1.57075 -1.57" xyz="${big_wheel_back_x} ${right_wheel_y} ${big_wheel_z}"/>
+    <origin xyz="${big_wheel_back_x} ${right_wheel_y} ${big_wheel_z}" rpy="0 1.57075 -1.57"/>
   </joint>
   <link name="right_wheel_big_back">
     <visual>
-      <origin rpy="0 0 0" xyz="0 0 0"/>
+      <origin xyz="0 0 0" rpy="0 0 0"/>
       <geometry>
         <cylinder length="${wheel_length}" radius="${wheel_radius}"/>
@@ -323,12 +323,12 @@
   </link>
   <joint name="left_crawler_joint" type="fixed">
-    <axis rpy="0 0 0" xyz="0 0 -1"/>
+    <axis xyz="0 0 -1" rpy="0 0 0"/>
     <parent link="base_body"/>
     <child link="left_crawler"/>
-    <origin rpy="0 1.57075 -1.57" xyz="-0.01 0.22 -0.043"/>
+    <origin xyz="-0.01 0.22 -0.043" rpy="0 1.57075 -1.57"/>
   </joint>
   <link name="left_crawler">
     <visual>
-      <origin rpy="0 0 0" xyz="0 0 0"/>
+      <origin xyz="0 0 0" rpy="0 0 0"/>
       <geometry>
         <mesh filename="file://$(find cugo_ros2_control)/models/cugo/meshes/cugo_v3_l-CuGoV3_L001.stl" scale="0.001 0.001 0.001"/>
@@ -342,12 +342,12 @@
   </link>
   <joint name="right_crawler_joint" type="fixed">
-    <axis rpy="0 0 0" xyz="0 0 -1"/>
+    <axis xyz="0 0 -1" rpy="0 0 0"/>
     <parent link="base_body"/>
     <child link="right_crawler"/>
-    <origin rpy="0 1.57075 -1.57" xyz="-0.10 -0.2065 -0.055"/>
+    <origin xyz="-0.10 -0.2065 -0.055" rpy="0 1.57075 -1.57"/>
   </joint>
   <link name="right_crawler">
     <visual>
-      <origin rpy="0 0 0" xyz="0 0 0"/>
+      <origin xyz="0 0 0" rpy="0 0 0"/>
       <geometry>
         <mesh filename="file://$(find cugo_ros2_control)/models/cugo/meshes/cugo_v3_r-CuGoV3_R001.stl" scale="0.001 0.001 0.001"/>
