Commit message: urdfのジョイントのトルク制限を調整し、速度制限を追加

File: models/cugo/cugo.urdf (robot description, URDF)
Before this commit: robot cugo_v3, 16 links, 15 joints
Joints:
- joint left_wheel_joint: limit (none) -> lower=-1.57 upper=1.57 effort=1.0 velocity=2.0
- joint left_wheel_joint_big_back: limit (none) -> lower=-1.57 upper=1.57 effort=1.0 velocity=2.0
- joint left_wheel_joint_big_front: limit (none) -> lower=-1.57 upper=1.57 effort=1.0 velocity=2.0
- joint left_wheel_joint_center_mini_back: limit (none) -> lower=-1.57 upper=1.57 effort=1.0 velocity=2.0
- joint left_wheel_joint_center_mini_front: limit (none) -> lower=-1.57 upper=1.57 effort=1.0 velocity=2.0
- joint right_wheel_joint: limit (none) -> lower=-1.57 upper=1.57 effort=0.5 velocity=2.0
- joint right_wheel_joint_big_back: limit (none) -> lower=-1.57 upper=1.57 effort=1.0 velocity=2.0
- joint right_wheel_joint_big_front: limit (none) -> lower=-1.57 upper=1.57 effort=1.0 velocity=2.0
- joint right_wheel_joint_center_mini_back: limit (none) -> lower=-1.57 upper=1.57 effort=1.0 velocity=2.0
- joint right_wheel_joint_center_mini_front: limit (none) -> lower=-1.57 upper=1.57 effort=1.0 velocity=2.0

File: models/cugo/cugo.xacro (robot description, xacro)
@@ -62,4 +62,5 @@
   <joint name="right_wheel_joint" type="continuous">
     <axis rpy="0 0 0" xyz="0 0 -1"/>
+    <limit lower="-1.57" upper="1.57" effort="0.5" velocity="2.0"/>
     <parent link="base_body"/>
     <child link="right_wheel"/>
@@ -98,4 +99,5 @@
   <joint name="right_wheel_joint_center_mini_front" type="continuous">
     <axis rpy="0 0 0" xyz="0 0 -1"/>
+    <limit lower="-1.57" upper="1.57" effort="1.0" velocity="2.0"/>
     <parent link="base_body"/>
     <child link="right_wheel_center_mini_front"/>
@@ -130,4 +132,5 @@
   <joint name="right_wheel_joint_center_mini_back" type="continuous">
     <axis rpy="0 0 0" xyz="0 0 -1"/>
+    <limit lower="-1.57" upper="1.57" effort="1.0" velocity="2.0"/>
     <parent link="base_body"/>
     <child link="right_wheel_center_mini_back"/>
@@ -214,4 +217,5 @@
   <joint name="right_wheel_joint_big_front" type="continuous">
     <axis rpy="0 0 0" xyz="0 0 -1"/>
+    <limit lower="-1.57" upper="1.57" effort="1.0" velocity="2.0"/>
     <parent link="base_body"/>
     <child link="right_wheel_big_front"/>
@@ -246,4 +250,5 @@
   <joint name="right_wheel_joint_big_back" type="continuous">
     <axis rpy="0 0 0" xyz="0 0 -1"/>
+    <limit lower="-1.57" upper="1.57" effort="1.0" velocity="2.0"/>
     <parent link="base_body"/>
     <child link="right_wheel_big_back"/>
@@ -278,4 +283,5 @@
   <joint name="left_wheel_joint" type="continuous">
     <axis rpy="0 0 0" xyz="0 0 -1"/>
+    <limit lower="-1.57" upper="1.57" effort="1.0" velocity="2.0"/>
     <parent link="base_body"/>
     <child link="left_wheel"/>
@@ -314,4 +320,5 @@
   <joint name="left_wheel_joint_center_mini_front" type="continuous">
     <axis rpy="0 0 0" xyz="0 0 -1"/>
+    <limit lower="-1.57" upper="1.57" effort="1.0" velocity="2.0"/>
     <parent link="base_body"/>
     <child link="left_wheel_center_mini_front"/>
@@ -346,4 +353,5 @@
   <joint name="left_wheel_joint_center_mini_back" type="continuous">
     <axis rpy="0 0 0" xyz="0 0 -1"/>
+    <limit lower="-1.57" upper="1.57" effort="1.0" velocity="2.0"/>
     <parent link="base_body"/>
     <child link="left_wheel_center_mini_back"/>
@@ -430,4 +438,5 @@
   <joint name="left_wheel_joint_big_front" type="continuous">
     <axis rpy="0 0 0" xyz="0 0 -1"/>
+    <limit lower="-1.57" upper="1.57" effort="1.0" velocity="2.0"/>
     <parent link="base_body"/>
     <child link="left_wheel_big_front"/>
@@ -461,4 +470,5 @@
   <joint name="left_wheel_joint_big_back" type="continuous">
     <axis rpy="0 0 0" xyz="0 0 -1"/>
+    <limit lower="-1.57" upper="1.57" effort="1.0" velocity="2.0"/>
     <parent link="base_body"/>
     <child link="left_wheel_big_back"/>
@@ -589,8 +599,8 @@
     <!--<plugin name="differential_drive_controller" filename="libgazebo_ros_diff_drive.so">-->
     <plugin name="cugo_diff_drive" filename="libgazebo_ros_diff_drive.so">
-      <update_rate>30</update_rate>
+      <update_rate>10</update_rate>
       <!-- wheels -->
-      <left_joint>left_wheel_joint</left_joint>
-      <right_joint>right_wheel_joint</right_joint>
+      <left_joint>right_wheel_joint</left_joint>
+      <right_joint>left_wheel_joint</right_joint>
       <!-- kinematics -->
       <wheel_separation>0.460</wheel_separation>
@@ -598,5 +608,5 @@
       <!-- limits -->
       <max_wheel_acceleration>1.0</max_wheel_acceleration>
-      <max_wheel_torque>20</max_wheel_torque>
+      <max_wheel_torque>1.0</max_wheel_torque>
       <command_topic>cmd_vel</command_topic>
       <!-- output -->
@@ -615,13 +625,15 @@
   <gazebo>
     <plugin name="cugo_diff_drive_mini_front" filename="libgazebo_ros_diff_drive.so">
-      <left_joint>left_wheel_joint_center_mini_front</left_joint>
-      <right_joint>right_wheel_joint_center_mini_front</right_joint>
-      <!--<robotBaseFrame>base_link</robotBaseFrame>-->
+      <update_rate>10</update_rate>
+      <!-- wheels -->
+      <left_joint>right_wheel_joint_center_mini_front</left_joint>
+      <right_joint>left_wheel_joint_center_mini_front</right_joint>
+      <!-- kinematics -->
       <wheel_separation>0.460</wheel_separation>
       <wheel_diameter>0.040</wheel_diameter>
-      <updateRate>10</updateRate>
-      <wheelAcceleration>1.0</wheelAcceleration>
-      <wheelTorque>20</wheelTorque>
-      <commandTopic>cmd_vel</commandTopic>
+      <!-- limits -->
+      <max_wheel_acceleration>1.0</max_wheel_acceleration>
+      <max_wheel_torque>1.0</max_wheel_torque>
+      <command_topic>cmd_vel</command_topic>
        <!--
       <odometryTopic>odom</odometryTopic>
@@ -637,13 +649,15 @@
   <gazebo>
     <plugin name="cugo_diff_drive_mini_back" filename="libgazebo_ros_diff_drive.so">
-      <left_joint>left_wheel_joint_center_mini_back</left_joint>
-      <right_joint>right_wheel_joint_center_mini_back</right_joint>
-      <!--<robotBaseFrame>base_link</robotBaseFrame>-->
-      <wheel_separation>0.460</wheel_separation>
+      <update_rate>10</update_rate>
+      <!-- wheels -->
+      <left_joint>right_wheel_joint_center_mini_back</left_joint>
+      <right_joint>left_wheel_joint_center_mini_back</right_joint>
+      <!-- kinematics -->
+      <wheel_separation>0.160</wheel_separation>
       <wheel_diameter>0.040</wheel_diameter>
-      <updateRate>10</updateRate>
-      <wheelAcceleration>1.0</wheelAcceleration>
-      <wheelTorque>20</wheelTorque>
-      <commandTopic>cmd_vel</commandTopic>
+      <!-- limits -->
+      <max_wheel_acceleration>1.0</max_wheel_acceleration>
+      <max_wheel_torque>1.0</max_wheel_torque>
+      <command_topic>cmd_vel</command_topic>
       <!--
       <odometryTopic>odom</odometryTopic>
@@ -659,13 +673,15 @@
   <gazebo>
     <plugin name="cugo_diff_drive_big_front" filename="libgazebo_ros_diff_drive.so">
-      <left_joint>left_wheel_joint_big_front</left_joint>
-      <right_joint>right_wheel_joint_big_front</right_joint>
-      <!--<robotBaseFrame>base_link</robotBaseFrame>-->
+      <update_rate>10</update_rate>
+      <!-- wheels -->
+      <left_joint>right_wheel_joint_big_front</left_joint>
+      <right_joint>left_wheel_joint_big_front</right_joint>
+      <!-- kinematics -->
       <wheel_separation>0.460</wheel_separation>
       <wheel_diameter>0.050</wheel_diameter>
-      <updateRate>10</updateRate>
-      <wheelAcceleration>1.0</wheelAcceleration>
-      <wheelTorque>20</wheelTorque>
-      <commandTopic>cmd_vel</commandTopic>
+      <!-- limits -->
+      <max_wheel_acceleration>1.0</max_wheel_acceleration>
+      <max_wheel_torque>1.0</max_wheel_torque>
+      <command_topic>cmd_vel</command_topic>
       <!--
       <odometryTopic>odom</odometryTopic>
@@ -681,13 +697,15 @@
   <gazebo>
     <plugin name="cugo_diff_drive_big_back" filename="libgazebo_ros_diff_drive.so">
-      <left_joint>left_wheel_joint_big_back</left_joint>
-      <right_joint>right_wheel_joint_big_back</right_joint>
-      <!--<robotBaseFrame>base_link</robotBaseFrame>-->
+      <update_rate>10</update_rate>
+      <!-- wheels -->
+      <left_joint>right_wheel_joint_big_back</left_joint>
+      <right_joint>left_wheel_joint_big_back</right_joint>
+      <!-- kinematics -->
       <wheel_separation>0.460</wheel_separation>
       <wheel_diameter>0.050</wheel_diameter>
-      <updateRate>10</updateRate>
-      <wheelAcceleration>1.0</wheelAcceleration>
-      <wheelTorque>20</wheelTorque>
-      <commandTopic>cmd_vel</commandTopic>
+      <!-- limits -->
+      <max_wheel_acceleration>1.0</max_wheel_acceleration>
+      <max_wheel_torque>1.0</max_wheel_torque>
+      <command_topic>cmd_vel</command_topic>
       <!--
       <odometryTopic>odom</odometryTopic>

Commit message: urdfに当たり判定の箱を追加

File: models/cugo/cugo.urdf (robot description, URDF)
Before this commit: robot cugo_v3, 16 links, 15 joints
Links:
- added link tbox, mass 0.1; collision box size=0.42 0.58 0.2; visual box size=0.42 0.58 0.2
Joints:
- added joint tbox_body: type fixed, parent base_body, child tbox, origin xyz=0 0 0.18 rpy=0 0 0

File: models/cugo/cugo.xacro (robot description, xacro)
@@ -6,4 +6,7 @@
   <xacro:property name="body_depth" value="0.58" />
   <xacro:property name="body_height" value="0.26" />
+  <xacro:property name="tbox_width" value="0.42" />
+  <xacro:property name="tbox_depth" value="0.58" />
+  <xacro:property name="tbox_height" value="0.20" />
   <xacro:property name="wheel_length" value="0.06" />
   <!--<xacro:property name="wheel_length" value="0.145" />-->
@@ -52,4 +55,28 @@
         <mesh filename="file://$(find cugo_ros2_control)/urdf/xacro/roskit-Compound.dae" scale="1 1 1"/>
     -->
+      </geometry>
+    </collision>
+    <inertial>
+      <mass value="0.1"/>
+      <inertia ixx="0.13542" iyy="0.10833" izz="0.17708" ixy="0.0" ixz="0.0" iyz="0.0"/>
+    </inertial>
+  </link>
+  <joint name="tbox_body" type="fixed">
+    <parent link="base_body"/>
+    <child link="tbox"/>
+    <origin rpy="0 0 0" xyz="0 0 ${tbox_height/2+body_height/2-0.05}"/>
+  </joint>
+  <!-- タカチボックス -->
+  <link name="tbox">
+    <visual>
+      <geometry>
+        <box size="${tbox_width} ${tbox_depth} ${tbox_height}"/>
+      </geometry>
+      <origin xyz="0 0 0" rpy="0 0 0"/>
+      <material name="white"/>
+    </visual>
+    <collision>
+      <geometry>
+        <box size="${tbox_width} ${tbox_depth} ${tbox_height}"/>
       </geometry>
     </collision>
