Commit message: cugo.xacroの不要なコメントを削除

File: models/cugo/cugo.urdf (robot description, URDF)
Before this commit: robot cugo_v3, 17 links, 16 joints
Links:
- removed link tbox
- added link body_collision, mass 0.1; collision box size=0.42 0.58 0.2; visual box size=0.42 0.58 0.2
Joints:
- removed joint tbox_body
- added joint body_collision_joint: type fixed, parent base_body, child body_collision, origin xyz=0 0 0.18 rpy=0 0 0

File: models/cugo/cugo.xacro (robot description, xacro)
@@ -9,13 +9,12 @@
   <xacro:property name="tbox_depth" value="0.58" />
   <xacro:property name="tbox_height" value="0.20" />
+  <xacro:property name="body_collision_width" value="0.42" />
+  <xacro:property name="body_collision_depth" value="0.58" />
+  <xacro:property name="body_collision_height" value="0.20" />
   <xacro:property name="wheel_length" value="0.06" />
-  <!--<xacro:property name="wheel_length" value="0.145" />-->
   <xacro:property name="collision_wheel_length" value="0.145" />
-  <!-- これは本当の車輪径 -->
-  <!-- <xacro:property name="wheel_radius" value="0.03858" /> -->
   <!-- 当たり判定の径 -->
   <xacro:property name="wheel_radius" value="0.050" />
   <!-- スプロケット径 -->
-  <!-- <xacro:property name="mini_wheel_radius" value="0.01929" /> -->
   <xacro:property name="mini_wheel_radius" value="0.040" />
   <xacro:property name="big_wheel_front_y" value="0.167" />
@@ -31,5 +30,4 @@
     <origin xyz="0.0 0.0 0.1065" rpy="0 0 0"/>
   </joint>
-  <!-- base_link -->
   <link name="base_link"/>
   <joint name="body_joint" type="fixed">
@@ -38,11 +36,7 @@
     <origin rpy="0 0 0" xyz="0 0 0"/>
   </joint>
-  <!-- 箱 -->
   <link name="base_body">
     <visual>
       <geometry>
-        <!--<box size="0.58 0.58 0.3"/>-->
-        <!--<box size="${body_depth} ${body_width} ${body_height}"/>-->
-        <!--<mesh filename="file://$(find cugo_ros2_control)/urdf/xacro/roskit-Compound.dae" scale="1 1 1"/>-->
         <mesh filename="file://$(find cugo_ros2_control)/models/cugo/meshes/roskit-Compound.dae" scale="1 1 1"/>
       </geometry>
@@ -50,11 +44,4 @@
       <material name="red"/>
     </visual>
-    <collision>
-      <geometry>
-    <!--
-        <mesh filename="file://$(find cugo_ros2_control)/urdf/xacro/roskit-Compound.dae" scale="1 1 1"/>
-    -->
-      </geometry>
-    </collision>
     <inertial>
       <mass value="0.1"/>
@@ -62,567 +49,317 @@
     </inertial>
   </link>
-  <joint name="tbox_body" type="fixed">
-    <parent link="base_body"/>
-    <child link="tbox"/>
-    <origin rpy="0 0 0" xyz="0 0 ${tbox_height/2+body_height/2-0.05}"/>
-  </joint>
-  <!-- タカチボックス -->
-  <link name="tbox">
-    <visual>
-      <geometry>
-        <box size="${tbox_width} ${tbox_depth} ${tbox_height}"/>
+  <joint name="body_collision_joint" type="fixed">
+    <parent link="base_body"/>
+    <child link="body_collision"/>
+    <origin rpy="0 0 0" xyz="0 0 ${body_collision_height/2+body_height/2-0.05}"/>
+  </joint>
+  <link name="body_collision">
+    <visual>
+      <geometry>
+        <box size="${body_collision_width} ${body_collision_depth} ${body_collision_height}"/>
       </geometry>
       <origin xyz="0 0 0" rpy="0 0 0"/>
+      <material name="dummy_white"/>
+    </visual>
+    <collision>
+      <geometry>
+        <box size="${body_collision_width} ${body_collision_depth} ${body_collision_height}"/>
+      </geometry>
+    </collision>
+    <inertial>
+      <mass value="0.1"/>
+      <inertia ixx="0.13542" iyy="0.10833" izz="0.17708" ixy="0.0" ixz="0.0" iyz="0.0"/>
+    </inertial>
+  </link>
+  <joint name="right_wheel_joint" type="continuous">
+    <axis rpy="0 0 0" xyz="0 0 -1"/>
+    <limit lower="-1.57" upper="1.57" effort="0.5" velocity="2.0"/>
+    <parent link="base_body"/>
+    <child link="right_wheel"/>
+    <origin rpy="0 1.57075 -1.57" xyz="0 ${right_wheel_x} ${center_wheel_z}"/>
+  </joint>
+  <link name="right_wheel">
+    <visual>
+      <origin rpy="0 0 0" xyz="0 0 0"/>
+      <geometry>
+        <cylinder length="${wheel_length}" radius="${mini_wheel_radius}"/>
+      </geometry>
+      <material name="dummy_white"/>
+    </visual>
+    <collision>
+      <geometry>
+        <cylinder length="${collision_wheel_length}" radius="${mini_wheel_radius}"/>
+      </geometry>
+    </collision>
+    <inertial>
+      <mass value="0.1"/>
+      <inertia ixx="0.00024" iyy="0.00024" izz="0.00015" ixy="0.0" ixz="0.0" iyz="0.0"/>
+    </inertial>
+  </link>
+  <joint name="right_wheel_joint_center_mini_front" type="continuous">
+    <axis rpy="0 0 0" xyz="0 0 -1"/>
+    <limit lower="-1.57" upper="1.57" effort="1.0" velocity="2.0"/>
+    <parent link="base_body"/>
+    <child link="right_wheel_center_mini_front"/>
+    <origin rpy="0 1.57075 -1.57" xyz="${mini_wheel_radius*2} ${right_wheel_x} ${center_wheel_z}"/>
+  </joint>
+  <link name="right_wheel_center_mini_front">
+    <visual>
+      <origin rpy="0 0 0" xyz="0 0 0"/>
+      <geometry>
+        <cylinder length="${wheel_length}" radius="${mini_wheel_radius}"/>
+      </geometry>
+      <material name="dummy_white"/>
+    </visual>
+    <collision>
+      <geometry>
+        <cylinder length="${collision_wheel_length}" radius="${mini_wheel_radius}"/>
+      </geometry>
+    </collision>
+    <inertial>
+      <mass value="0.1"/>
+      <inertia ixx="0.00024" iyy="0.00024" izz="0.00015" ixy="0.0" ixz="0.0" iyz="0.0"/>
+    </inertial>
+  </link>
+  <joint name="right_wheel_joint_center_mini_back" type="continuous">
+    <axis rpy="0 0 0" xyz="0 0 -1"/>
+    <limit lower="-1.57" upper="1.57" effort="1.0" velocity="2.0"/>
+    <parent link="base_body"/>
+    <child link="right_wheel_center_mini_back"/>
+    <origin rpy="0 1.57075 -1.57" xyz="-${mini_wheel_radius*2} ${right_wheel_x} ${center_wheel_z}"/>
+  </joint>
+  <link name="right_wheel_center_mini_back">
+    <visual>
+      <origin rpy="0 0 0" xyz="0 0 0"/>
+      <geometry>
+        <cylinder length="${wheel_length}" radius="${mini_wheel_radius}"/>
+      </geometry>
+      <material name="dummy_white"/>
+    </visual>
+    <collision>
+      <geometry>
+        <cylinder length="${collision_wheel_length}" radius="${mini_wheel_radius}"/>
+      </geometry>
+    </collision>
+    <inertial>
+      <mass value="0.1"/>
+      <inertia ixx="0.00024" iyy="0.00024" izz="0.00015" ixy="0.0" ixz="0.0" iyz="0.0"/>
+    </inertial>
+  </link>
+  <joint name="right_wheel_joint_big_front" type="continuous">
+    <axis rpy="0 0 0" xyz="0 0 -1"/>
+    <limit lower="-1.57" upper="1.57" effort="1.0" velocity="2.0"/>
+    <parent link="base_body"/>
+    <child link="right_wheel_big_front"/>
+    <origin rpy="0 1.57075 -1.57" xyz="${big_wheel_front_y} ${right_wheel_x} ${big_wheel_z}"/>
+  </joint>
+  <link name="right_wheel_big_front">
+    <visual>
+      <origin rpy="0 0 0" xyz="0 0 0"/>
+      <geometry>
+        <cylinder length="${wheel_length}" radius="${wheel_radius}"/>
+      </geometry>
+      <material name="dummy_white"/>
+    </visual>
+    <collision>
+      <geometry>
+        <cylinder length="${collision_wheel_length}" radius="${wheel_radius}"/>
+      </geometry>
+    </collision>
+    <inertial>
+      <mass value="0.1"/>
+      <inertia ixx="0.00024" iyy="0.00024" izz="0.00015" ixy="0.0" ixz="0.0" iyz="0.0"/>
+    </inertial>
+  </link>
+  <joint name="right_wheel_joint_big_back" type="continuous">
+    <axis rpy="0 0 0" xyz="0 0 -1"/>
+    <limit lower="-1.57" upper="1.57" effort="1.0" velocity="2.0"/>
+    <parent link="base_body"/>
+    <child link="right_wheel_big_back"/>
+    <origin rpy="0 1.57075 -1.57" xyz="${big_wheel_back_y} ${right_wheel_x} ${big_wheel_z}"/>
+  </joint>
+  <link name="right_wheel_big_back">
+    <visual>
+      <origin rpy="0 0 0" xyz="0 0 0"/>
+      <geometry>
+        <cylinder length="${wheel_length}" radius="${wheel_radius}"/>
+      </geometry>
+      <material name="dummy_white"/>
+    </visual>
+    <collision>
+      <geometry>
+        <cylinder length="${collision_wheel_length}" radius="${wheel_radius}"/>
+      </geometry>
+    </collision>
+    <inertial>
+      <mass value="0.1"/>
+      <inertia ixx="0.00024" iyy="0.00024" izz="0.00015" ixy="0.0" ixz="0.0" iyz="0.0"/>
+    </inertial>
+  </link>
+  <joint name="left_wheel_joint" type="continuous">
+    <axis rpy="0 0 0" xyz="0 0 -1"/>
+    <limit lower="-1.57" upper="1.57" effort="1.0" velocity="2.0"/>
+    <parent link="base_body"/>
+    <child link="left_wheel"/>
+    <origin rpy="0 1.57075 -1.57" xyz="0 ${left_wheel_x} ${center_wheel_z}"/>
+  </joint>
+  <link name="left_wheel">
+    <visual>
+      <origin rpy="0 0 0" xyz="0 0 0"/>
+      <geometry>
+        <cylinder length="${wheel_length}" radius="${mini_wheel_radius}"/>
+      </geometry>
+      <material name="dummy_white"/>
+    </visual>
+    <collision>
+      <geometry>
+        <cylinder length="${collision_wheel_length}" radius="${mini_wheel_radius}"/>
+      </geometry>
+    </collision>
+    <inertial>
+      <mass value="0.1"/>
+      <inertia ixx="0.00024" iyy="0.00024" izz="0.00015" ixy="0.0" ixz="0.0" iyz="0.0"/>
+    </inertial>
+  </link>
+  <joint name="left_wheel_joint_center_mini_front" type="continuous">
+    <axis rpy="0 0 0" xyz="0 0 -1"/>
+    <limit lower="-1.57" upper="1.57" effort="1.0" velocity="2.0"/>
+    <parent link="base_body"/>
+    <child link="left_wheel_center_mini_front"/>
+    <origin rpy="0 1.57075 -1.57" xyz="${mini_wheel_radius*2} ${left_wheel_x} ${center_wheel_z}"/>
+  </joint>
+  <link name="left_wheel_center_mini_front">
+    <visual>
+      <origin rpy="0 0 0" xyz="0 0 0"/>
+      <geometry>
+        <cylinder length="${wheel_length}" radius="${mini_wheel_radius}"/>
+      </geometry>
+      <material name="dummy_white"/>
+    </visual>
+    <collision>
+      <geometry>
+        <cylinder length="${collision_wheel_length}" radius="${mini_wheel_radius}"/>
+      </geometry>
+    </collision>
+    <inertial>
+      <mass value="0.1"/>
+      <inertia ixx="0.00024" iyy="0.00024" izz="0.00015" ixy="0.0" ixz="0.0" iyz="0.0"/>
+    </inertial>
+  </link>
+  <joint name="left_wheel_joint_center_mini_back" type="continuous">
+    <axis rpy="0 0 0" xyz="0 0 -1"/>
+    <limit lower="-1.57" upper="1.57" effort="1.0" velocity="2.0"/>
+    <parent link="base_body"/>
+    <child link="left_wheel_center_mini_back"/>
+    <origin rpy="0 1.57075 -1.57" xyz="-${mini_wheel_radius*2} ${left_wheel_x} ${center_wheel_z}"/>
+  </joint>
+  <link name="left_wheel_center_mini_back">
+    <visual>
+      <origin rpy="0 0 0" xyz="0 0 0"/>
+      <geometry>
+        <cylinder length="${wheel_length}" radius="${mini_wheel_radius}"/>
+      </geometry>
+      <material name="dummy_white"/>
+    </visual>
+    <collision>
+      <geometry>
+        <cylinder length="${collision_wheel_length}" radius="${mini_wheel_radius}"/>
+      </geometry>
+    </collision>
+    <inertial>
+      <mass value="0.1"/>
+      <inertia ixx="0.00024" iyy="0.00024" izz="0.00015" ixy="0.0" ixz="0.0" iyz="0.0"/>
+    </inertial>
+  </link>
+  <joint name="left_wheel_joint_big_front" type="continuous">
+    <axis rpy="0 0 0" xyz="0 0 -1"/>
+    <limit lower="-1.57" upper="1.57" effort="1.0" velocity="2.0"/>
+    <parent link="base_body"/>
+    <child link="left_wheel_big_front"/>
+    <origin rpy="0 1.57075 -1.57" xyz="${big_wheel_front_y} ${left_wheel_x} ${big_wheel_z}"/>
+  </joint>
+  <link name="left_wheel_big_front">
+    <visual>
+      <origin rpy="0 0 0" xyz="0 0 0"/>
+      <geometry>
+        <cylinder length="${wheel_length}" radius="${wheel_radius}"/>
+      </geometry>
+      <material name="dummy_white"/>
+    </visual>
+    <collision>
+      <geometry>
+        <cylinder length="${collision_wheel_length}" radius="${wheel_radius}"/>
+      </geometry>
+    </collision>
+    <inertial>
+      <mass value="0.1"/>
+      <inertia ixx="0.00024" iyy="0.00024" izz="0.00015" ixy="0.0" ixz="0.0" iyz="0.0"/>
+    </inertial>
+  </link>
+  <joint name="left_wheel_joint_big_back" type="continuous">
+    <axis rpy="0 0 0" xyz="0 0 -1"/>
+    <limit lower="-1.57" upper="1.57" effort="1.0" velocity="2.0"/>
+    <parent link="base_body"/>
+    <child link="left_wheel_big_back"/>
+    <origin rpy="0 1.57075 -1.57" xyz="${big_wheel_back_y} ${left_wheel_x} ${big_wheel_z}"/>
+  </joint>
+  <link name="left_wheel_big_back">
+    <visual>
+      <origin rpy="0 0 0" xyz="0 0 0"/>
+      <geometry>
+        <cylinder length="${wheel_length}" radius="${wheel_radius}"/>
+      </geometry>
+      <material name="dummy_white"/>
+    </visual>
+    <collision>
+      <geometry>
+        <cylinder length="${collision_wheel_length}" radius="${wheel_radius}"/>
+      </geometry>
+    </collision>
+    <inertial>
+      <mass value="0.1"/>
+      <inertia ixx="0.00024" iyy="0.00024" izz="0.00015" ixy="0.0" ixz="0.0" iyz="0.0"/>
+    </inertial>
+  </link>
+  <joint name="right_crawler_joint" type="fixed">
+    <axis rpy="0 0 0" xyz="0 0 -1"/>
+    <parent link="base_body"/>
+    <child link="right_crawler"/>
+    <origin rpy="0 1.57075 -1.57" xyz="-0.01 0.22 -0.043"/>
+  </joint>
+  <link name="right_crawler">
+    <visual>
+      <origin rpy="0 0 0" xyz="0 0 0"/>
+      <geometry>
+        <mesh filename="file://$(find cugo_ros2_control)/models/cugo/meshes/cugo_v3_l-CuGoV3_L001.stl" scale="0.001 0.001 0.001"/>
+      </geometry>
       <material name="white"/>
     </visual>
-    <collision>
-      <geometry>
-        <box size="${tbox_width} ${tbox_depth} ${tbox_height}"/>
-      </geometry>
-    </collision>
-    <inertial>
-      <mass value="0.1"/>
-      <inertia ixx="0.13542" iyy="0.10833" izz="0.17708" ixy="0.0" ixz="0.0" iyz="0.0"/>
-    </inertial>
-  </link>
-  <!-- 車輪のジョイントと車輪のリンク -->
-  <joint name="right_wheel_joint" type="continuous">
-    <axis rpy="0 0 0" xyz="0 0 -1"/>
-    <limit lower="-1.57" upper="1.57" effort="0.5" velocity="2.0"/>
-    <parent link="base_body"/>
-    <child link="right_wheel"/>
-    <!--<origin rpy="0 0 0" xyz="-0.133333333333 0 -0.085"/>-->
-    <!--<origin rpy="0 1.57075 0" xyz="0.230 0 -0.1"/>-->
-    <!--<origin rpy="0 1.57075 0" xyz="0.115 0 -0.16142"/>-->
-    <!--<origin rpy="0 1.57075 0" xyz="0.1 0 -0.13858"/>-->
-    <!--<origin rpy="0 1.57075 0" xyz="0.2055 0 -0.178935"/>-->
-    <!--<origin rpy="0 1.57075 0" xyz="0.2055 0 -0.215"/>-->
-    <!--<origin rpy="0 1.57075 0" xyz="${right_wheel_x} 0 ${center_wheel_z}"/>-->
-    <origin rpy="0 1.57075 -1.57" xyz="0 ${right_wheel_x} ${center_wheel_z}"/>
-  </joint>
-  <link name="right_wheel">
-    <visual>
-      <!--<origin rpy="1.57075 0 0" xyz="0 0 0"/>-->
-      <origin rpy="0 0 0" xyz="0 0 0"/>
-      <geometry>
-        <!--<cylinder length="0.1" radius="0.03858"/>-->
-        <!--<cylinder length="0.169" radius="0.01929"/>-->
-        <cylinder length="${wheel_length}" radius="${mini_wheel_radius}"/>
-      </geometry>
-      <material name="dummy_white"/>
-    </visual>
-    <collision>
-      <geometry>
-        <!--<cylinder length="0.1" radius="0.03858"/>-->
-        <!--<cylinder length="0.169" radius="0.01929"/>-->
-        <cylinder length="${collision_wheel_length}" radius="${mini_wheel_radius}"/>
-      </geometry>
-    </collision>
-    <inertial>
-      <mass value="0.1"/>
-      <inertia ixx="0.00024" iyy="0.00024" izz="0.00015" ixy="0.0" ixz="0.0" iyz="0.0"/>
-    </inertial>
-  </link>
-  <joint name="right_wheel_joint_center_mini_front" type="continuous">
-    <axis rpy="0 0 0" xyz="0 0 -1"/>
-    <limit lower="-1.57" upper="1.57" effort="1.0" velocity="2.0"/>
-    <parent link="base_body"/>
-    <child link="right_wheel_center_mini_front"/>
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