Commit message: cugo.xacroの左右逆だったジョイント名を修正

File: models/cugo/cugo.urdf (robot description, URDF)
Before this commit: robot cugo_v3, 17 links, 16 joints
Joints:
- joint left_crawler_joint: origin xyz=-0.10 -0.2065 -0.055 rpy=0 1.57075 -1.57 -> xyz=-0.01 0.22 -0.043 rpy=0 1.57075 -1.57
- joint left_wheel_joint: limit lower=-1.57 upper=1.57 effort=1.0 velocity=2.0 -> lower=-1.57 upper=1.57 effort=0.5 velocity=2.0; origin xyz=0 -0.22 -0.105 rpy=0 1.57075 -1.57 -> xyz=0 0.24 -0.105 rpy=0 1.57075 -1.57
- joint left_wheel_joint_big_back: origin xyz=-0.167 -0.22 -0.08 rpy=0 1.57075 -1.57 -> xyz=-0.167 0.24 -0.08 rpy=0 1.57075 -1.57
- joint left_wheel_joint_big_front: origin xyz=0.167 -0.22 -0.08 rpy=0 1.57075 -1.57 -> xyz=0.167 0.24 -0.08 rpy=0 1.57075 -1.57
- joint left_wheel_joint_center_mini_back: origin xyz=-0.08 -0.22 -0.105 rpy=0 1.57075 -1.57 -> xyz=-0.08 0.24 -0.105 rpy=0 1.57075 -1.57
- joint left_wheel_joint_center_mini_front: origin xyz=0.08 -0.22 -0.105 rpy=0 1.57075 -1.57 -> xyz=0.08 0.24 -0.105 rpy=0 1.57075 -1.57
- joint right_crawler_joint: origin xyz=-0.01 0.22 -0.043 rpy=0 1.57075 -1.57 -> xyz=-0.10 -0.2065 -0.055 rpy=0 1.57075 -1.57
- joint right_wheel_joint: limit lower=-1.57 upper=1.57 effort=0.5 velocity=2.0 -> lower=-1.57 upper=1.57 effort=1.0 velocity=2.0; origin xyz=0 0.24 -0.105 rpy=0 1.57075 -1.57 -> xyz=0 -0.22 -0.105 rpy=0 1.57075 -1.57
- joint right_wheel_joint_big_back: origin xyz=-0.167 0.24 -0.08 rpy=0 1.57075 -1.57 -> xyz=-0.167 -0.22 -0.08 rpy=0 1.57075 -1.57
- joint right_wheel_joint_big_front: origin xyz=0.167 0.24 -0.08 rpy=0 1.57075 -1.57 -> xyz=0.167 -0.22 -0.08 rpy=0 1.57075 -1.57
- joint right_wheel_joint_center_mini_back: origin xyz=-0.08 0.24 -0.105 rpy=0 1.57075 -1.57 -> xyz=-0.08 -0.22 -0.105 rpy=0 1.57075 -1.57
- joint right_wheel_joint_center_mini_front: origin xyz=0.08 0.24 -0.105 rpy=0 1.57075 -1.57 -> xyz=0.08 -0.22 -0.105 rpy=0 1.57075 -1.57

File: models/cugo/cugo.xacro (robot description, xacro)
@@ -18,10 +18,10 @@
   <!-- スプロケット径 -->
   <xacro:property name="mini_wheel_radius" value="0.040" />
-  <xacro:property name="big_wheel_front_y" value="0.167" />
-  <xacro:property name="big_wheel_back_y" value="-0.167" />
+  <xacro:property name="big_wheel_front_x" value="0.167" />
+  <xacro:property name="big_wheel_back_x" value="-0.167" />
   <xacro:property name="center_wheel_z" value="-0.105" />
   <xacro:property name="big_wheel_z" value="-0.08" />
-  <xacro:property name="right_wheel_x" value="0.24" />
-  <xacro:property name="left_wheel_x" value="-0.22" />
+  <xacro:property name="left_wheel_y" value="0.24" />
+  <xacro:property name="right_wheel_y" value="-0.22" />
   <link name="base_footprint"/>
   <joint name="base_footprint_joint" type="fixed">
@@ -72,10 +72,135 @@
     </inertial>
   </link>
+  <joint name="left_wheel_joint" type="continuous">
+    <axis rpy="0 0 0" xyz="0 0 -1"/>
+    <limit lower="-1.57" upper="1.57" effort="0.5" velocity="2.0"/>
+    <parent link="base_body"/>
+    <child link="left_wheel"/>
+    <origin rpy="0 1.57075 -1.57" xyz="0 ${left_wheel_y} ${center_wheel_z}"/>
+  </joint>
+  <link name="left_wheel">
+    <visual>
+      <origin rpy="0 0 0" xyz="0 0 0"/>
+      <geometry>
+        <cylinder length="${wheel_length}" radius="${mini_wheel_radius}"/>
+      </geometry>
+      <material name="dummy_white"/>
+    </visual>
+    <collision>
+      <geometry>
+        <cylinder length="${collision_wheel_length}" radius="${mini_wheel_radius}"/>
+      </geometry>
+    </collision>
+    <inertial>
+      <mass value="0.1"/>
+      <inertia ixx="0.00024" iyy="0.00024" izz="0.00015" ixy="0.0" ixz="0.0" iyz="0.0"/>
+    </inertial>
+  </link>
+  <joint name="left_wheel_joint_center_mini_front" type="continuous">
+    <axis rpy="0 0 0" xyz="0 0 -1"/>
+    <limit lower="-1.57" upper="1.57" effort="1.0" velocity="2.0"/>
+    <parent link="base_body"/>
+    <child link="left_wheel_center_mini_front"/>
+    <origin rpy="0 1.57075 -1.57" xyz="${mini_wheel_radius*2} ${left_wheel_y} ${center_wheel_z}"/>
+  </joint>
+  <link name="left_wheel_center_mini_front">
+    <visual>
+      <origin rpy="0 0 0" xyz="0 0 0"/>
+      <geometry>
+        <cylinder length="${wheel_length}" radius="${mini_wheel_radius}"/>
+      </geometry>
+      <material name="dummy_white"/>
+    </visual>
+    <collision>
+      <geometry>
+        <cylinder length="${collision_wheel_length}" radius="${mini_wheel_radius}"/>
+      </geometry>
+    </collision>
+    <inertial>
+      <mass value="0.1"/>
+      <inertia ixx="0.00024" iyy="0.00024" izz="0.00015" ixy="0.0" ixz="0.0" iyz="0.0"/>
+    </inertial>
+  </link>
+  <joint name="left_wheel_joint_center_mini_back" type="continuous">
+    <axis rpy="0 0 0" xyz="0 0 -1"/>
+    <limit lower="-1.57" upper="1.57" effort="1.0" velocity="2.0"/>
+    <parent link="base_body"/>
+    <child link="left_wheel_center_mini_back"/>
+    <origin rpy="0 1.57075 -1.57" xyz="-${mini_wheel_radius*2} ${left_wheel_y} ${center_wheel_z}"/>
+  </joint>
+  <link name="left_wheel_center_mini_back">
+    <visual>
+      <origin rpy="0 0 0" xyz="0 0 0"/>
+      <geometry>
+        <cylinder length="${wheel_length}" radius="${mini_wheel_radius}"/>
+      </geometry>
+      <material name="dummy_white"/>
+    </visual>
+    <collision>
+      <geometry>
+        <cylinder length="${collision_wheel_length}" radius="${mini_wheel_radius}"/>
+      </geometry>
+    </collision>
+    <inertial>
+      <mass value="0.1"/>
+      <inertia ixx="0.00024" iyy="0.00024" izz="0.00015" ixy="0.0" ixz="0.0" iyz="0.0"/>
+    </inertial>
+  </link>
+  <joint name="left_wheel_joint_big_front" type="continuous">
+    <axis rpy="0 0 0" xyz="0 0 -1"/>
+    <limit lower="-1.57" upper="1.57" effort="1.0" velocity="2.0"/>
+    <parent link="base_body"/>
+    <child link="left_wheel_big_front"/>
+    <origin rpy="0 1.57075 -1.57" xyz="${big_wheel_front_x} ${left_wheel_y} ${big_wheel_z}"/>
+  </joint>
+  <link name="left_wheel_big_front">
+    <visual>
+      <origin rpy="0 0 0" xyz="0 0 0"/>
+      <geometry>
+        <cylinder length="${wheel_length}" radius="${wheel_radius}"/>
+      </geometry>
+      <material name="dummy_white"/>
+    </visual>
+    <collision>
+      <geometry>
+        <cylinder length="${collision_wheel_length}" radius="${wheel_radius}"/>
+      </geometry>
+    </collision>
+    <inertial>
+      <mass value="0.1"/>
+      <inertia ixx="0.00024" iyy="0.00024" izz="0.00015" ixy="0.0" ixz="0.0" iyz="0.0"/>
+    </inertial>
+  </link>
+  <joint name="left_wheel_joint_big_back" type="continuous">
+    <axis rpy="0 0 0" xyz="0 0 -1"/>
+    <limit lower="-1.57" upper="1.57" effort="1.0" velocity="2.0"/>
+    <parent link="base_body"/>
+    <child link="left_wheel_big_back"/>
+    <origin rpy="0 1.57075 -1.57" xyz="${big_wheel_back_x} ${left_wheel_y} ${big_wheel_z}"/>
+  </joint>
+  <link name="left_wheel_big_back">
+    <visual>
+      <origin rpy="0 0 0" xyz="0 0 0"/>
+      <geometry>
+        <cylinder length="${wheel_length}" radius="${wheel_radius}"/>
+      </geometry>
+      <material name="dummy_white"/>
+    </visual>
+    <collision>
+      <geometry>
+        <cylinder length="${collision_wheel_length}" radius="${wheel_radius}"/>
+      </geometry>
+    </collision>
+    <inertial>
+      <mass value="0.1"/>
+      <inertia ixx="0.00024" iyy="0.00024" izz="0.00015" ixy="0.0" ixz="0.0" iyz="0.0"/>
+    </inertial>
+  </link>
   <joint name="right_wheel_joint" type="continuous">
     <axis rpy="0 0 0" xyz="0 0 -1"/>
-    <limit lower="-1.57" upper="1.57" effort="0.5" velocity="2.0"/>
+    <limit lower="-1.57" upper="1.57" effort="1.0" velocity="2.0"/>
     <parent link="base_body"/>
     <child link="right_wheel"/>
-    <origin rpy="0 1.57075 -1.57" xyz="0 ${right_wheel_x} ${center_wheel_z}"/>
+    <origin rpy="0 1.57075 -1.57" xyz="0 ${right_wheel_y} ${center_wheel_z}"/>
   </joint>
   <link name="right_wheel">
@@ -102,5 +227,5 @@
     <parent link="base_body"/>
     <child link="right_wheel_center_mini_front"/>
-    <origin rpy="0 1.57075 -1.57" xyz="${mini_wheel_radius*2} ${right_wheel_x} ${center_wheel_z}"/>
+    <origin rpy="0 1.57075 -1.57" xyz="${mini_wheel_radius*2} ${right_wheel_y} ${center_wheel_z}"/>
   </joint>
   <link name="right_wheel_center_mini_front">
@@ -127,5 +252,5 @@
     <parent link="base_body"/>
     <child link="right_wheel_center_mini_back"/>
-    <origin rpy="0 1.57075 -1.57" xyz="-${mini_wheel_radius*2} ${right_wheel_x} ${center_wheel_z}"/>
+    <origin rpy="0 1.57075 -1.57" xyz="-${mini_wheel_radius*2} ${right_wheel_y} ${center_wheel_z}"/>
   </joint>
   <link name="right_wheel_center_mini_back">
@@ -152,5 +277,5 @@
     <parent link="base_body"/>
     <child link="right_wheel_big_front"/>
-    <origin rpy="0 1.57075 -1.57" xyz="${big_wheel_front_y} ${right_wheel_x} ${big_wheel_z}"/>
+    <origin rpy="0 1.57075 -1.57" xyz="${big_wheel_front_x} ${right_wheel_y} ${big_wheel_z}"/>
   </joint>
   <link name="right_wheel_big_front">
@@ -177,5 +302,5 @@
     <parent link="base_body"/>
     <child link="right_wheel_big_back"/>
-    <origin rpy="0 1.57075 -1.57" xyz="${big_wheel_back_y} ${right_wheel_x} ${big_wheel_z}"/>
+    <origin rpy="0 1.57075 -1.57" xyz="${big_wheel_back_x} ${right_wheel_y} ${big_wheel_z}"/>
   </joint>
   <link name="right_wheel_big_back">
@@ -197,124 +322,18 @@
     </inertial>
   </link>
-  <joint name="left_wheel_joint" type="continuous">
-    <axis rpy="0 0 0" xyz="0 0 -1"/>
-    <limit lower="-1.57" upper="1.57" effort="1.0" velocity="2.0"/>
-    <parent link="base_body"/>
-    <child link="left_wheel"/>
-    <origin rpy="0 1.57075 -1.57" xyz="0 ${left_wheel_x} ${center_wheel_z}"/>
-  </joint>
-  <link name="left_wheel">
-    <visual>
-      <origin rpy="0 0 0" xyz="0 0 0"/>
-      <geometry>
-        <cylinder length="${wheel_length}" radius="${mini_wheel_radius}"/>
-      </geometry>
-      <material name="dummy_white"/>
-    </visual>
-    <collision>
-      <geometry>
-        <cylinder length="${collision_wheel_length}" radius="${mini_wheel_radius}"/>
-      </geometry>
-    </collision>
-    <inertial>
-      <mass value="0.1"/>
-      <inertia ixx="0.00024" iyy="0.00024" izz="0.00015" ixy="0.0" ixz="0.0" iyz="0.0"/>
-    </inertial>
-  </link>
-  <joint name="left_wheel_joint_center_mini_front" type="continuous">
-    <axis rpy="0 0 0" xyz="0 0 -1"/>
-    <limit lower="-1.57" upper="1.57" effort="1.0" velocity="2.0"/>
-    <parent link="base_body"/>
-    <child link="left_wheel_center_mini_front"/>
-    <origin rpy="0 1.57075 -1.57" xyz="${mini_wheel_radius*2} ${left_wheel_x} ${center_wheel_z}"/>
-  </joint>
-  <link name="left_wheel_center_mini_front">
-    <visual>
-      <origin rpy="0 0 0" xyz="0 0 0"/>
-      <geometry>
-        <cylinder length="${wheel_length}" radius="${mini_wheel_radius}"/>
-      </geometry>
-      <material name="dummy_white"/>
-    </visual>
-    <collision>
-      <geometry>
-        <cylinder length="${collision_wheel_length}" radius="${mini_wheel_radius}"/>
-      </geometry>
-    </collision>
-    <inertial>
-      <mass value="0.1"/>
-      <inertia ixx="0.00024" iyy="0.00024" izz="0.00015" ixy="0.0" ixz="0.0" iyz="0.0"/>
-    </inertial>
-  </link>
-  <joint name="left_wheel_joint_center_mini_back" type="continuous">
-    <axis rpy="0 0 0" xyz="0 0 -1"/>
-    <limit lower="-1.57" upper="1.57" effort="1.0" velocity="2.0"/>
-    <parent link="base_body"/>
-    <child link="left_wheel_center_mini_back"/>
-    <origin rpy="0 1.57075 -1.57" xyz="-${mini_wheel_radius*2} ${left_wheel_x} ${center_wheel_z}"/>
-  </joint>
-  <link name="left_wheel_center_mini_back">
-    <visual>
-      <origin rpy="0 0 0" xyz="0 0 0"/>
-      <geometry>
-        <cylinder length="${wheel_length}" radius="${mini_wheel_radius}"/>
-      </geometry>
-      <material name="dummy_white"/>
-    </visual>
-    <collision>
-      <geometry>
-        <cylinder length="${collision_wheel_length}" radius="${mini_wheel_radius}"/>
-      </geometry>
-    </collision>
-    <inertial>
-      <mass value="0.1"/>
-      <inertia ixx="0.00024" iyy="0.00024" izz="0.00015" ixy="0.0" ixz="0.0" iyz="0.0"/>
-    </inertial>
-  </link>
-  <joint name="left_wheel_joint_big_front" type="continuous">
-    <axis rpy="0 0 0" xyz="0 0 -1"/>
-    <limit lower="-1.57" upper="1.57" effort="1.0" velocity="2.0"/>
-    <parent link="base_body"/>
-    <child link="left_wheel_big_front"/>
-    <origin rpy="0 1.57075 -1.57" xyz="${big_wheel_front_y} ${left_wheel_x} ${big_wheel_z}"/>
-  </joint>
-  <link name="left_wheel_big_front">
-    <visual>
-      <origin rpy="0 0 0" xyz="0 0 0"/>
-      <geometry>
-        <cylinder length="${wheel_length}" radius="${wheel_radius}"/>
-      </geometry>
-      <material name="dummy_white"/>
-    </visual>
-    <collision>
-      <geometry>
-        <cylinder length="${collision_wheel_length}" radius="${wheel_radius}"/>
-      </geometry>
-    </collision>
-    <inertial>
-      <mass value="0.1"/>
-      <inertia ixx="0.00024" iyy="0.00024" izz="0.00015" ixy="0.0" ixz="0.0" iyz="0.0"/>
-    </inertial>
-  </link>
-  <joint name="left_wheel_joint_big_back" type="continuous">
-    <axis rpy="0 0 0" xyz="0 0 -1"/>
-    <limit lower="-1.57" upper="1.57" effort="1.0" velocity="2.0"/>
-    <parent link="base_body"/>
-    <child link="left_wheel_big_back"/>
-    <origin rpy="0 1.57075 -1.57" xyz="${big_wheel_back_y} ${left_wheel_x} ${big_wheel_z}"/>
-  </joint>
-  <link name="left_wheel_big_back">
-    <visual>
-      <origin rpy="0 0 0" xyz="0 0 0"/>
-      <geometry>
-        <cylinder length="${wheel_length}" radius="${wheel_radius}"/>
-      </geometry>
-      <material name="dummy_white"/>
-    </visual>
-    <collision>
-      <geometry>
-        <cylinder length="${collision_wheel_length}" radius="${wheel_radius}"/>
-      </geometry>
-    </collision>
+  <joint name="left_crawler_joint" type="fixed">
+    <axis rpy="0 0 0" xyz="0 0 -1"/>
+    <parent link="base_body"/>
+    <child link="left_crawler"/>
+    <origin rpy="0 1.57075 -1.57" xyz="-0.01 0.22 -0.043"/>
+  </joint>
+  <link name="left_crawler">
+    <visual>
+      <origin rpy="0 0 0" xyz="0 0 0"/>
+      <geometry>
+        <mesh filename="file://$(find cugo_ros2_control)/models/cugo/meshes/cugo_v3_l-CuGoV3_L001.stl" scale="0.001 0.001 0.001"/>
+      </geometry>
+      <material name="white"/>
+    </visual>
     <inertial>
       <mass value="0.1"/>
@@ -326,26 +345,7 @@
     <parent link="base_body"/>
     <child link="right_crawler"/>
-    <origin rpy="0 1.57075 -1.57" xyz="-0.01 0.22 -0.043"/>
+    <origin rpy="0 1.57075 -1.57" xyz="-0.10 -0.2065 -0.055"/>
   </joint>
   <link name="right_crawler">
-    <visual>
-      <origin rpy="0 0 0" xyz="0 0 0"/>
-      <geometry>
-        <mesh filename="file://$(find cugo_ros2_control)/models/cugo/meshes/cugo_v3_l-CuGoV3_L001.stl" scale="0.001 0.001 0.001"/>
-      </geometry>
-      <material name="white"/>
-    </visual>
-    <inertial>
-      <mass value="0.1"/>
-      <inertia ixx="0.00024" iyy="0.00024" izz="0.00015" ixy="0.0" ixz="0.0" iyz="0.0"/>
-    </inertial>
-  </link>
-  <joint name="left_crawler_joint" type="fixed">
-    <axis rpy="0 0 0" xyz="0 0 -1"/>
-    <parent link="base_body"/>
-    <child link="left_crawler"/>
-    <origin rpy="0 1.57075 -1.57" xyz="-0.10 -0.2065 -0.055"/>
-  </joint>
-  <link name="left_crawler">
     <visual>
       <origin rpy="0 0 0" xyz="0 0 0"/>
@@ -365,6 +365,6 @@
       <update_rate>10</update_rate>
       <!-- wheels -->
-      <left_joint>right_wheel_joint</left_joint>
-      <right_joint>left_wheel_joint</right_joint>
+      <left_joint>left_wheel_joint</left_joint>
+      <right_joint>right_wheel_joint</right_joint>
       <!-- kinematics -->
       <wheel_separation>0.460</wheel_separation>
@@ -391,6 +391,6 @@
       <update_rate>10</update_rate>
       <!-- wheels -->
-      <left_joint>right_wheel_joint_center_mini_front</left_joint>
-      <right_joint>left_wheel_joint_center_mini_front</right_joint>
+      <left_joint>left_wheel_joint_center_mini_front</left_joint>
+      <right_joint>right_wheel_joint_center_mini_front</right_joint>
       <!-- kinematics -->
       <wheel_separation>0.460</wheel_separation>
@@ -407,6 +407,6 @@
       <update_rate>10</update_rate>
       <!-- wheels -->
-      <left_joint>right_wheel_joint_center_mini_back</left_joint>
-      <right_joint>left_wheel_joint_center_mini_back</right_joint>
+      <left_joint>left_wheel_joint_center_mini_back</left_joint>
+      <right_joint>right_wheel_joint_center_mini_back</right_joint>
       <!-- kinematics -->
       <wheel_separation>0.160</wheel_separation>
@@ -423,6 +423,6 @@
       <update_rate>10</update_rate>
       <!-- wheels -->
-      <left_joint>right_wheel_joint_big_front</left_joint>
-      <right_joint>left_wheel_joint_big_front</right_joint>
+      <left_joint>left_wheel_joint_big_front</left_joint>
+      <right_joint>right_wheel_joint_big_front</right_joint>
       <!-- kinematics -->
       <wheel_separation>0.460</wheel_separation>
@@ -439,6 +439,6 @@
       <update_rate>10</update_rate>
       <!-- wheels -->
-      <left_joint>right_wheel_joint_big_back</left_joint>
-      <right_joint>left_wheel_joint_big_back</right_joint>
+      <left_joint>left_wheel_joint_big_back</left_joint>
+      <right_joint>right_wheel_joint_big_back</right_joint>
       <!-- kinematics -->
       <wheel_separation>0.460</wheel_separation>
