Commit message: xacroにて車輪径をすべて同じ径に統一

File: models/cugo/cugo.urdf (robot description, URDF)
Before this commit: robot cugo_v3, 17 links, 16 joints
Links:
- link left_wheel: geometry collision cylinder length=0.145 radius=0.03858; visual cylinder length=0.06 radius=0.03858
- link left_wheel_big_back: geometry collision cylinder length=0.145 radius=0.03858; visual cylinder length=0.06 radius=0.03858
- link left_wheel_big_front: geometry collision cylinder length=0.145 radius=0.03858; visual cylinder length=0.06 radius=0.03858
- link left_wheel_center_mini_back: geometry collision cylinder length=0.145 radius=0.03858; visual cylinder length=0.06 radius=0.03858
- link left_wheel_center_mini_front: geometry collision cylinder length=0.145 radius=0.03858; visual cylinder length=0.06 radius=0.03858
- link right_wheel: geometry collision cylinder length=0.145 radius=0.03858; visual cylinder length=0.06 radius=0.03858
- link right_wheel_big_back: geometry collision cylinder length=0.145 radius=0.03858; visual cylinder length=0.06 radius=0.03858
- link right_wheel_big_front: geometry collision cylinder length=0.145 radius=0.03858; visual cylinder length=0.06 radius=0.03858
- link right_wheel_center_mini_back: geometry collision cylinder length=0.145 radius=0.03858; visual cylinder length=0.06 radius=0.03858
- link right_wheel_center_mini_front: geometry collision cylinder length=0.145 radius=0.03858; visual cylinder length=0.06 radius=0.03858
Joints:
- joint left_wheel_joint_big_back: origin xyz=-0.167 0.24 -0.08 rpy=0 1.57075 -1.57 -> xyz=-0.172 0.24 -0.08 rpy=0 1.57075 -1.57
- joint left_wheel_joint_big_front: origin xyz=0.167 0.24 -0.08 rpy=0 1.57075 -1.57 -> xyz=0.172 0.24 -0.08 rpy=0 1.57075 -1.57
- joint left_wheel_joint_center_mini_back: origin xyz=-0.08 0.24 -0.105 rpy=0 1.57075 -1.57 -> xyz=-0.07716 0.24 -0.105 rpy=0 1.57075 -1.57
- joint left_wheel_joint_center_mini_front: origin xyz=0.08 0.24 -0.105 rpy=0 1.57075 -1.57 -> xyz=0.07716 0.24 -0.105 rpy=0 1.57075 -1.57
- joint right_wheel_joint_big_back: origin xyz=-0.167 -0.22 -0.08 rpy=0 1.57075 -1.57 -> xyz=-0.172 -0.22 -0.08 rpy=0 1.57075 -1.57
- joint right_wheel_joint_big_front: origin xyz=0.167 -0.22 -0.08 rpy=0 1.57075 -1.57 -> xyz=0.172 -0.22 -0.08 rpy=0 1.57075 -1.57
- joint right_wheel_joint_center_mini_back: origin xyz=-0.08 -0.22 -0.105 rpy=0 1.57075 -1.57 -> xyz=-0.07716 -0.22 -0.105 rpy=0 1.57075 -1.57
- joint right_wheel_joint_center_mini_front: origin xyz=0.08 -0.22 -0.105 rpy=0 1.57075 -1.57 -> xyz=0.07716 -0.22 -0.105 rpy=0 1.57075 -1.57

File: models/cugo/cugo.xacro (robot description, xacro)
@@ -15,9 +15,12 @@
   <xacro:property name="collision_wheel_length" value="0.145" />
   <!-- 当たり判定の径 -->
-  <xacro:property name="wheel_radius" value="0.050" />
+  <xacro:property name="wheel_radius" value="0.03858" />
   <!-- スプロケット径 -->
-  <xacro:property name="mini_wheel_radius" value="0.040" />
-  <xacro:property name="big_wheel_front_x" value="0.167" />
-  <xacro:property name="big_wheel_back_x" value="-0.167" />
+  <xacro:property name="mini_wheel_radius" value="0.03858" />
+  <xacro:property name="wheel_diameter" value="0.07716" />
+  <xacro:property name="max_wheel_acceleration" value="1.0" />
+  <xacro:property name="max_wheel_torque" value="5.0" />
+  <xacro:property name="big_wheel_front_x" value="0.172" />
+  <xacro:property name="big_wheel_back_x" value="-0.172" />
   <xacro:property name="center_wheel_z" value="-0.105" />
   <xacro:property name="big_wheel_z" value="-0.08" />
@@ -369,8 +372,8 @@
       <!-- kinematics -->
       <wheel_separation>0.460</wheel_separation>
-      <wheel_diameter>0.040</wheel_diameter>
+      <wheel_diameter>${wheel_diameter}</wheel_diameter>
       <!-- limits -->
-      <max_wheel_acceleration>1.0</max_wheel_acceleration>
-      <max_wheel_torque>1.0</max_wheel_torque>
+      <max_wheel_acceleration>${max_wheel_acceleration}</max_wheel_acceleration>
+      <max_wheel_torque>${max_wheel_torque}</max_wheel_torque>
       <command_topic>cmd_vel</command_topic>
       <!-- output -->
@@ -395,8 +398,8 @@
       <!-- kinematics -->
       <wheel_separation>0.460</wheel_separation>
-      <wheel_diameter>0.040</wheel_diameter>
+      <wheel_diameter>${wheel_diameter}</wheel_diameter>
       <!-- limits -->
-      <max_wheel_acceleration>1.0</max_wheel_acceleration>
-      <max_wheel_torque>1.0</max_wheel_torque>
+      <max_wheel_acceleration>${max_wheel_acceleration}</max_wheel_acceleration>
+      <max_wheel_torque>${max_wheel_torque}</max_wheel_torque>
       <command_topic>cmd_vel</command_topic>
       <legacyMode>false</legacyMode>
@@ -410,9 +413,9 @@
       <right_joint>right_wheel_joint_center_mini_back</right_joint>
       <!-- kinematics -->
-      <wheel_separation>0.160</wheel_separation>
-      <wheel_diameter>0.040</wheel_diameter>
+      <wheel_separation>0.460</wheel_separation>
+      <wheel_diameter>${wheel_diameter}</wheel_diameter>
       <!-- limits -->
-      <max_wheel_acceleration>1.0</max_wheel_acceleration>
-      <max_wheel_torque>1.0</max_wheel_torque>
+      <max_wheel_acceleration>${max_wheel_acceleration}</max_wheel_acceleration>
+      <max_wheel_torque>${max_wheel_torque}</max_wheel_torque>
       <command_topic>cmd_vel</command_topic>
       <legacyMode>false</legacyMode>
@@ -427,8 +430,8 @@
       <!-- kinematics -->
       <wheel_separation>0.460</wheel_separation>
-      <wheel_diameter>0.050</wheel_diameter>
+      <wheel_diameter>${wheel_diameter}</wheel_diameter>
       <!-- limits -->
-      <max_wheel_acceleration>1.0</max_wheel_acceleration>
-      <max_wheel_torque>1.0</max_wheel_torque>
+      <max_wheel_acceleration>${max_wheel_acceleration}</max_wheel_acceleration>
+      <max_wheel_torque>${max_wheel_torque}</max_wheel_torque>
       <command_topic>cmd_vel</command_topic>
       <legacyMode>false</legacyMode>
@@ -443,8 +446,8 @@
       <!-- kinematics -->
       <wheel_separation>0.460</wheel_separation>
-      <wheel_diameter>0.050</wheel_diameter>
+      <wheel_diameter>${wheel_diameter}</wheel_diameter>
       <!-- limits -->
-      <max_wheel_acceleration>1.0</max_wheel_acceleration>
-      <max_wheel_torque>1.0</max_wheel_torque>
+      <max_wheel_acceleration>${max_wheel_acceleration}</max_wheel_acceleration>
+      <max_wheel_torque>${max_wheel_torque}</max_wheel_torque>
       <command_topic>cmd_vel</command_topic>
       <legacyMode>false</legacyMode>
