Commit message: xacroのリンク名、ジョイント名を修正

File: models/cugo_v3/cugo_v3.urdf (robot description, URDF)
Before this commit: robot cugo_v3, 17 links, 16 joints
Links:
- removed link left_wheel
- removed link left_wheel_big_back
- removed link left_wheel_big_front
- removed link left_wheel_center_mini_back
- removed link left_wheel_center_mini_front
- removed link right_wheel
- removed link right_wheel_big_back
- removed link right_wheel_big_front
- removed link right_wheel_center_mini_back
- removed link right_wheel_center_mini_front
- added link left_back_wheel, mass 0.1; collision cylinder length=0.145 radius=0.03858; visual cylinder length=0.06 radius=0.03858
- added link left_center_1_wheel, mass 0.1; collision cylinder length=0.145 radius=0.03858; visual cylinder length=0.06 radius=0.03858
- added link left_center_2_wheel, mass 0.1; collision cylinder length=0.145 radius=0.03858; visual cylinder length=0.06 radius=0.03858
- added link left_center_3_wheel, mass 0.1; collision cylinder length=0.145 radius=0.03858; visual cylinder length=0.06 radius=0.03858
- added link left_front_wheel, mass 0.1; collision cylinder length=0.145 radius=0.03858; visual cylinder length=0.06 radius=0.03858
- added link right_back_wheel, mass 0.1; collision cylinder length=0.145 radius=0.03858; visual cylinder length=0.06 radius=0.03858
- added link right_center_1_wheel, mass 0.1; collision cylinder length=0.145 radius=0.03858; visual cylinder length=0.06 radius=0.03858
- added link right_center_2_wheel, mass 0.1; collision cylinder length=0.145 radius=0.03858; visual cylinder length=0.06 radius=0.03858
- added link right_center_3_wheel, mass 0.1; collision cylinder length=0.145 radius=0.03858; visual cylinder length=0.06 radius=0.03858
- added link right_front_wheel, mass 0.1; collision cylinder length=0.145 radius=0.03858; visual cylinder length=0.06 radius=0.03858
Joints:
- removed joint base_footprint_joint
- removed joint left_wheel_joint
- removed joint left_wheel_joint_big_back
- removed joint left_wheel_joint_big_front
- removed joint left_wheel_joint_center_mini_back
- removed joint left_wheel_joint_center_mini_front
- removed joint right_wheel_joint
- removed joint right_wheel_joint_big_back
- removed joint right_wheel_joint_big_front
- removed joint right_wheel_joint_center_mini_back
- removed joint right_wheel_joint_center_mini_front
- added joint base_joint: type fixed, parent base_footprint, child base_link, origin xyz=0.0 0.0 0.1065 rpy=0 0 0
- added joint left_back_wheel_joint: type continuous, parent base_body, child left_back_wheel, origin xyz=-0.172 0.24 -0.08 rpy=0 1.57075 -1.57, axis 0 0 -1, limit lower=-1.57 upper=1.57 effort=1.0 velocity=2.0
- added joint left_center_1_wheel_joint: type continuous, parent base_body, child left_center_1_wheel, origin xyz=0.07716 0.24 -0.105 rpy=0 1.57075 -1.57, axis 0 0 -1, limit lower=-1.57 upper=1.57 effort=1.0 velocity=2.0
- added joint left_center_2_wheel_joint: type continuous, parent base_body, child left_center_2_wheel, origin xyz=0 0.24 -0.105 rpy=0 1.57075 -1.57, axis 0 0 -1, limit lower=-1.57 upper=1.57 effort=0.5 velocity=2.0
- added joint left_center_3_wheel_joint: type continuous, parent base_body, child left_center_3_wheel, origin xyz=-0.07716 0.24 -0.105 rpy=0 1.57075 -1.57, axis 0 0 -1, limit lower=-1.57 upper=1.57 effort=1.0 velocity=2.0
- added joint left_front_wheel_joint: type continuous, parent base_body, child left_front_wheel, origin xyz=0.172 0.24 -0.08 rpy=0 1.57075 -1.57, axis 0 0 -1, limit lower=-1.57 upper=1.57 effort=1.0 velocity=2.0
- added joint right_back_wheel_joint: type continuous, parent base_body, child right_back_wheel, origin xyz=-0.172 -0.22 -0.08 rpy=0 1.57075 -1.57, axis 0 0 -1, limit lower=-1.57 upper=1.57 effort=1.0 velocity=2.0
- added joint right_center_1_wheel_joint: type continuous, parent base_body, child right_center_1_wheel, origin xyz=0.07716 -0.22 -0.105 rpy=0 1.57075 -1.57, axis 0 0 -1, limit lower=-1.57 upper=1.57 effort=1.0 velocity=2.0
- added joint right_center_2_wheel_joint: type continuous, parent base_body, child right_center_2_wheel, origin xyz=0 -0.22 -0.105 rpy=0 1.57075 -1.57, axis 0 0 -1, limit lower=-1.57 upper=1.57 effort=1.0 velocity=2.0
- added joint right_center_3_wheel_joint: type continuous, parent base_body, child right_center_3_wheel, origin xyz=-0.07716 -0.22 -0.105 rpy=0 1.57075 -1.57, axis 0 0 -1, limit lower=-1.57 upper=1.57 effort=1.0 velocity=2.0
- added joint right_front_wheel_joint: type continuous, parent base_body, child right_front_wheel, origin xyz=0.172 -0.22 -0.08 rpy=0 1.57075 -1.57, axis 0 0 -1, limit lower=-1.57 upper=1.57 effort=1.0 velocity=2.0

File: models/cugo_v3/cugo_v3.xacro (robot description, xacro)
@@ -28,5 +28,5 @@
   <xacro:property name="right_wheel_y" value="-0.22" />
   <link name="base_footprint"/>
-  <joint name="base_footprint_joint" type="fixed">
+  <joint name="base_joint" type="fixed">
     <parent link="base_footprint"/>
     <child link="base_link"/>
@@ -75,12 +75,12 @@
     </inertial>
   </link>
-  <joint name="left_wheel_joint" type="continuous">
+  <joint name="left_center_2_wheel_joint" type="continuous">
     <axis xyz="0 0 -1" rpy="0 0 0"/>
     <limit lower="-1.57" upper="1.57" effort="0.5" velocity="2.0"/>
     <parent link="base_body"/>
-    <child link="left_wheel"/>
+    <child link="left_center_2_wheel"/>
     <origin xyz="0 ${left_wheel_y} ${center_wheel_z}" rpy="0 1.57075 -1.57"/>
   </joint>
-  <link name="left_wheel">
+  <link name="left_center_2_wheel">
     <visual>
       <origin xyz="0 0 0" rpy="0 0 0"/>
@@ -100,12 +100,12 @@
     </inertial>
   </link>
-  <joint name="left_wheel_joint_center_mini_front" type="continuous">
-    <axis xyz="0 0 -1" rpy="0 0 0"/>
-    <limit lower="-1.57" upper="1.57" effort="1.0" velocity="2.0"/>
-    <parent link="base_body"/>
-    <child link="left_wheel_center_mini_front"/>
+  <joint name="left_center_1_wheel_joint" type="continuous">
+    <axis xyz="0 0 -1" rpy="0 0 0"/>
+    <limit lower="-1.57" upper="1.57" effort="1.0" velocity="2.0"/>
+    <parent link="base_body"/>
+    <child link="left_center_1_wheel"/>
     <origin xyz="${mini_wheel_radius*2} ${left_wheel_y} ${center_wheel_z}" rpy="0 1.57075 -1.57"/>
   </joint>
-  <link name="left_wheel_center_mini_front">
+  <link name="left_center_1_wheel">
     <visual>
       <origin xyz="0 0 0" rpy="0 0 0"/>
@@ -125,12 +125,12 @@
     </inertial>
   </link>
-  <joint name="left_wheel_joint_center_mini_back" type="continuous">
-    <axis xyz="0 0 -1" rpy="0 0 0"/>
-    <limit lower="-1.57" upper="1.57" effort="1.0" velocity="2.0"/>
-    <parent link="base_body"/>
-    <child link="left_wheel_center_mini_back"/>
+  <joint name="left_center_3_wheel_joint" type="continuous">
+    <axis xyz="0 0 -1" rpy="0 0 0"/>
+    <limit lower="-1.57" upper="1.57" effort="1.0" velocity="2.0"/>
+    <parent link="base_body"/>
+    <child link="left_center_3_wheel"/>
     <origin xyz="-${mini_wheel_radius*2} ${left_wheel_y} ${center_wheel_z}" rpy="0 1.57075 -1.57"/>
   </joint>
-  <link name="left_wheel_center_mini_back">
+  <link name="left_center_3_wheel">
     <visual>
       <origin xyz="0 0 0" rpy="0 0 0"/>
@@ -150,12 +150,12 @@
     </inertial>
   </link>
-  <joint name="left_wheel_joint_big_front" type="continuous">
-    <axis xyz="0 0 -1" rpy="0 0 0"/>
-    <limit lower="-1.57" upper="1.57" effort="1.0" velocity="2.0"/>
-    <parent link="base_body"/>
-    <child link="left_wheel_big_front"/>
+  <joint name="left_front_wheel_joint" type="continuous">
+    <axis xyz="0 0 -1" rpy="0 0 0"/>
+    <limit lower="-1.57" upper="1.57" effort="1.0" velocity="2.0"/>
+    <parent link="base_body"/>
+    <child link="left_front_wheel"/>
     <origin xyz="${big_wheel_front_x} ${left_wheel_y} ${big_wheel_z}" rpy="0 1.57075 -1.57"/>
   </joint>
-  <link name="left_wheel_big_front">
+  <link name="left_front_wheel">
     <visual>
       <origin xyz="0 0 0" rpy="0 0 0"/>
@@ -175,12 +175,12 @@
     </inertial>
   </link>
-  <joint name="left_wheel_joint_big_back" type="continuous">
-    <axis xyz="0 0 -1" rpy="0 0 0"/>
-    <limit lower="-1.57" upper="1.57" effort="1.0" velocity="2.0"/>
-    <parent link="base_body"/>
-    <child link="left_wheel_big_back"/>
+  <joint name="left_back_wheel_joint" type="continuous">
+    <axis xyz="0 0 -1" rpy="0 0 0"/>
+    <limit lower="-1.57" upper="1.57" effort="1.0" velocity="2.0"/>
+    <parent link="base_body"/>
+    <child link="left_back_wheel"/>
     <origin xyz="${big_wheel_back_x} ${left_wheel_y} ${big_wheel_z}" rpy="0 1.57075 -1.57"/>
   </joint>
-  <link name="left_wheel_big_back">
+  <link name="left_back_wheel">
     <visual>
       <origin xyz="0 0 0" rpy="0 0 0"/>
@@ -200,12 +200,12 @@
     </inertial>
   </link>
-  <joint name="right_wheel_joint" type="continuous">
-    <axis xyz="0 0 -1" rpy="0 0 0"/>
-    <limit lower="-1.57" upper="1.57" effort="1.0" velocity="2.0"/>
-    <parent link="base_body"/>
-    <child link="right_wheel"/>
+  <joint name="right_center_2_wheel_joint" type="continuous">
+    <axis xyz="0 0 -1" rpy="0 0 0"/>
+    <limit lower="-1.57" upper="1.57" effort="1.0" velocity="2.0"/>
+    <parent link="base_body"/>
+    <child link="right_center_2_wheel"/>
     <origin xyz="0 ${right_wheel_y} ${center_wheel_z}" rpy="0 1.57075 -1.57"/>
   </joint>
-  <link name="right_wheel">
+  <link name="right_center_2_wheel">
     <visual>
       <origin xyz="0 0 0" rpy="0 0 0"/>
@@ -225,12 +225,12 @@
     </inertial>
   </link>
-  <joint name="right_wheel_joint_center_mini_front" type="continuous">
-    <axis xyz="0 0 -1" rpy="0 0 0"/>
-    <limit lower="-1.57" upper="1.57" effort="1.0" velocity="2.0"/>
-    <parent link="base_body"/>
-    <child link="right_wheel_center_mini_front"/>
+  <joint name="right_center_1_wheel_joint" type="continuous">
+    <axis xyz="0 0 -1" rpy="0 0 0"/>
+    <limit lower="-1.57" upper="1.57" effort="1.0" velocity="2.0"/>
+    <parent link="base_body"/>
+    <child link="right_center_1_wheel"/>
     <origin xyz="${mini_wheel_radius*2} ${right_wheel_y} ${center_wheel_z}" rpy="0 1.57075 -1.57"/>
   </joint>
-  <link name="right_wheel_center_mini_front">
+  <link name="right_center_1_wheel">
     <visual>
       <origin xyz="0 0 0" rpy="0 0 0"/>
@@ -250,12 +250,12 @@
     </inertial>
   </link>
-  <joint name="right_wheel_joint_center_mini_back" type="continuous">
-    <axis xyz="0 0 -1" rpy="0 0 0"/>
-    <limit lower="-1.57" upper="1.57" effort="1.0" velocity="2.0"/>
-    <parent link="base_body"/>
-    <child link="right_wheel_center_mini_back"/>
+  <joint name="right_center_3_wheel_joint" type="continuous">
+    <axis xyz="0 0 -1" rpy="0 0 0"/>
+    <limit lower="-1.57" upper="1.57" effort="1.0" velocity="2.0"/>
+    <parent link="base_body"/>
+    <child link="right_center_3_wheel"/>
     <origin xyz="-${mini_wheel_radius*2} ${right_wheel_y} ${center_wheel_z}" rpy="0 1.57075 -1.57"/>
   </joint>
-  <link name="right_wheel_center_mini_back">
+  <link name="right_center_3_wheel">
     <visual>
       <origin xyz="0 0 0" rpy="0 0 0"/>
@@ -275,12 +275,12 @@
     </inertial>
   </link>
-  <joint name="right_wheel_joint_big_front" type="continuous">
-    <axis xyz="0 0 -1" rpy="0 0 0"/>
-    <limit lower="-1.57" upper="1.57" effort="1.0" velocity="2.0"/>
-    <parent link="base_body"/>
-    <child link="right_wheel_big_front"/>
+  <joint name="right_front_wheel_joint" type="continuous">
+    <axis xyz="0 0 -1" rpy="0 0 0"/>
+    <limit lower="-1.57" upper="1.57" effort="1.0" velocity="2.0"/>
+    <parent link="base_body"/>
+    <child link="right_front_wheel"/>
     <origin xyz="${big_wheel_front_x} ${right_wheel_y} ${big_wheel_z}" rpy="0 1.57075 -1.57"/>
   </joint>
-  <link name="right_wheel_big_front">
+  <link name="right_front_wheel">
     <visual>
       <origin xyz="0 0 0" rpy="0 0 0"/>
@@ -300,12 +300,12 @@
     </inertial>
   </link>
-  <joint name="right_wheel_joint_big_back" type="continuous">
-    <axis xyz="0 0 -1" rpy="0 0 0"/>
-    <limit lower="-1.57" upper="1.57" effort="1.0" velocity="2.0"/>
-    <parent link="base_body"/>
-    <child link="right_wheel_big_back"/>
+  <joint name="right_back_wheel_joint" type="continuous">
+    <axis xyz="0 0 -1" rpy="0 0 0"/>
+    <limit lower="-1.57" upper="1.57" effort="1.0" velocity="2.0"/>
+    <parent link="base_body"/>
+    <child link="right_back_wheel"/>
     <origin xyz="${big_wheel_back_x} ${right_wheel_y} ${big_wheel_z}" rpy="0 1.57075 -1.57"/>
   </joint>
-  <link name="right_wheel_big_back">
+  <link name="right_back_wheel">
     <visual>
       <origin xyz="0 0 0" rpy="0 0 0"/>
@@ -368,6 +368,6 @@
       <update_rate>10</update_rate>
       <!-- wheels -->
-      <left_joint>left_wheel_joint</left_joint>
-      <right_joint>right_wheel_joint</right_joint>
+      <left_joint>left_center_2_wheel_joint</left_joint>
+      <right_joint>right_center_2_wheel_joint</right_joint>
       <!-- kinematics -->
       <wheel_separation>0.460</wheel_separation>
@@ -394,6 +394,6 @@
       <update_rate>10</update_rate>
       <!-- wheels -->
-      <left_joint>left_wheel_joint_center_mini_front</left_joint>
-      <right_joint>right_wheel_joint_center_mini_front</right_joint>
+      <left_joint>left_center_1_wheel_joint</left_joint>
+      <right_joint>right_center_1_wheel_joint</right_joint>
       <!-- kinematics -->
       <wheel_separation>0.460</wheel_separation>
@@ -410,6 +410,6 @@
       <update_rate>10</update_rate>
       <!-- wheels -->
-      <left_joint>left_wheel_joint_center_mini_back</left_joint>
-      <right_joint>right_wheel_joint_center_mini_back</right_joint>
+      <left_joint>left_center_3_wheel_joint</left_joint>
+      <right_joint>right_center_3_wheel_joint</right_joint>
       <!-- kinematics -->
       <wheel_separation>0.460</wheel_separation>
@@ -426,6 +426,6 @@
       <update_rate>10</update_rate>
       <!-- wheels -->
-      <left_joint>left_wheel_joint_big_front</left_joint>
-      <right_joint>right_wheel_joint_big_front</right_joint>
+      <left_joint>left_front_wheel_joint</left_joint>
+      <right_joint>right_front_wheel_joint</right_joint>
       <!-- kinematics -->
       <wheel_separation>0.460</wheel_separation>
@@ -442,6 +442,6 @@
       <update_rate>10</update_rate>
       <!-- wheels -->
-      <left_joint>left_wheel_joint_big_back</left_joint>
-      <right_joint>right_wheel_joint_big_back</right_joint>
+      <left_joint>left_back_wheel_joint</left_joint>
+      <right_joint>right_back_wheel_joint</right_joint>
       <!-- kinematics -->
       <wheel_separation>0.460</wheel_separation>
@@ -455,44 +455,32 @@
   </gazebo>
   <!-- gazebo上のパーツ設定 -->
-  <xacro:gazebo_material ref="right_wheel" mu="2.0">
-    <material>Gazebo/GreyTransparent</material>
-  </xacro:gazebo_material>
-  <xacro:gazebo_material ref="right_wheel_center_mini_front" mu="2.0">
-    <material>Gazebo/GreyTransparent</material>
-  </xacro:gazebo_material>
-  <xacro:gazebo_material ref="right_wheel_center_mini_back" mu="2.0">
-    <material>Gazebo/GreyTransparent</material>
-  </xacro:gazebo_material>
-  <xacro:gazebo_material ref="right_wheel_mini_front" mu="2.0">
-    <material>Gazebo/GreyTransparent</material>
-  </xacro:gazebo_material>
-  <xacro:gazebo_material ref="right_wheel_mini_back" mu="2.0">
-    <material>Gazebo/GreyTransparent</material>
-  </xacro:gazebo_material>
-  <xacro:gazebo_material ref="right_wheel_big_front" mu="2.0">
-    <material>Gazebo/GreyTransparent</material>
-  </xacro:gazebo_material>
-  <xacro:gazebo_material ref="right_wheel_big_back" mu="2.0">
-    <material>Gazebo/GreyTransparent</material>
-  </xacro:gazebo_material>
-  <xacro:gazebo_material ref="left_wheel" mu="2.0">
-    <material>Gazebo/GreyTransparent</material>
-  </xacro:gazebo_material>
-  <xacro:gazebo_material ref="left_wheel_center_mini_front" mu="2.0">
-    <material>Gazebo/GreyTransparent</material>
-  </xacro:gazebo_material>
-  <xacro:gazebo_material ref="left_wheel_center_mini_back" mu="2.0">
-    <material>Gazebo/GreyTransparent</material>
-  </xacro:gazebo_material>
-  <xacro:gazebo_material ref="left_wheel_mini_front" mu="2.0">
-    <material>Gazebo/GreyTransparent</material>
-  </xacro:gazebo_material>
-  <xacro:gazebo_material ref="left_wheel_mini_back" mu="2.0">
-    <material>Gazebo/GreyTransparent</material>
-  </xacro:gazebo_material>
-  <xacro:gazebo_material ref="left_wheel_big_front" mu="2.0">
-    <material>Gazebo/GreyTransparent</material>
-  </xacro:gazebo_material>
-  <xacro:gazebo_material ref="left_wheel_big_back" mu="2.0">
+  <xacro:gazebo_material ref="right_center_2_wheel" mu="2.0">
+    <material>Gazebo/GreyTransparent</material>
+  </xacro:gazebo_material>
+  <xacro:gazebo_material ref="right_center_1_wheel" mu="2.0">
+    <material>Gazebo/GreyTransparent</material>
+  </xacro:gazebo_material>
+  <xacro:gazebo_material ref="right_center_3_wheel" mu="2.0">
+    <material>Gazebo/GreyTransparent</material>
+  </xacro:gazebo_material>
+  <xacro:gazebo_material ref="right_front_wheel" mu="2.0">
+    <material>Gazebo/GreyTransparent</material>
+  </xacro:gazebo_material>
+  <xacro:gazebo_material ref="right_back_wheel" mu="2.0">
+    <material>Gazebo/GreyTransparent</material>
+  </xacro:gazebo_material>
+  <xacro:gazebo_material ref="left_center_2_wheel" mu="2.0">
+    <material>Gazebo/GreyTransparent</material>
+  </xacro:gazebo_material>
+  <xacro:gazebo_material ref="left_center_1_wheel" mu="2.0">
+    <material>Gazebo/GreyTransparent</material>
+  </xacro:gazebo_material>
+  <xacro:gazebo_material ref="left_center_3_wheel" mu="2.0">
+    <material>Gazebo/GreyTransparent</material>
+  </xacro:gazebo_material>
+  <xacro:gazebo_material ref="left_front_wheel" mu="2.0">
+    <material>Gazebo/GreyTransparent</material>
+  </xacro:gazebo_material>
+  <xacro:gazebo_material ref="left_back_wheel" mu="2.0">
     <material>Gazebo/GreyTransparent</material>
   </xacro:gazebo_material>
