Commit message: urdf表示用launchファイルと、xacro, urdf内にあるモデルのファイルパスを修正

File: models/cugo_v3/cugo_v3.xacro (robot description, xacro)
@@ -1,6 +1,6 @@
 <?xml version="1.0"?>
 <robot xmlns:xacro="http://ros.org/wiki/xacro" name="cugo_v3">
-  <xacro:include filename="$(find cugo_ros2_control)/models/cugo/material_colors.xacro" />
-  <xacro:include filename="$(find cugo_ros2_control)/models/cugo/gazebo_material_macro.xacro" />
+  <xacro:include filename="$(find cugo_ros2_control)/models/cugo_v3/material_colors.xacro" />
+  <xacro:include filename="$(find cugo_ros2_control)/models/cugo_v3/gazebo_material_macro.xacro" />
   <xacro:property name="body_width" value="0.42" />
   <xacro:property name="body_depth" value="0.58" />
@@ -42,5 +42,5 @@
     <visual>
       <geometry>
-        <mesh filename="file://$(find cugo_ros2_control)/models/cugo/meshes/roskit-Compound.dae" scale="1 1 1"/>
+        <mesh filename="file://$(find cugo_ros2_control)/models/cugo_v3/meshes/roskit-Compound.dae" scale="1 1 1"/>
       </geometry>
       <origin xyz="0 0 0" rpy="0 0 -1.57"/>
@@ -335,5 +335,5 @@
       <origin xyz="0 0 0" rpy="0 0 0"/>
       <geometry>
-        <mesh filename="file://$(find cugo_ros2_control)/models/cugo/meshes/cugo_v3_l-CuGoV3_L001.stl" scale="0.001 0.001 0.001"/>
+        <mesh filename="file://$(find cugo_ros2_control)/models/cugo_v3/meshes/cugo_v3_l-CuGoV3_L001.stl" scale="0.001 0.001 0.001"/>
       </geometry>
       <material name="white"/>
@@ -354,5 +354,5 @@
       <origin xyz="0 0 0" rpy="0 0 0"/>
       <geometry>
-        <mesh filename="file://$(find cugo_ros2_control)/models/cugo/meshes/cugo_v3_r-CuGoV3_R001.stl" scale="0.001 0.001 0.001"/>
+        <mesh filename="file://$(find cugo_ros2_control)/models/cugo_v3/meshes/cugo_v3_r-CuGoV3_R001.stl" scale="0.001 0.001 0.001"/>
       </geometry>
       <material name="white"/>
@@ -510,5 +510,5 @@
       <origin xyz="0 0 0.0" rpy="0 0 -1.57"/>
       <geometry>
-        <mesh filename="file://$(find cugo_ros2_control)/models/cugo/meshes/lds.dae" scale="0.001 0.001 0.001"/>
+        <mesh filename="file://$(find cugo_ros2_control)/models/cugo_v3/meshes/lds.dae" scale="0.001 0.001 0.001"/>
       </geometry>
       <material name="dark"/>

Commit message: xacroのプロパティ名を修正

File: models/cugo_v3/cugo_v3.xacro (robot description, xacro)
@@ -12,19 +12,18 @@
   <xacro:property name="body_collision_depth" value="0.58" />
   <xacro:property name="body_collision_height" value="0.20" />
-  <xacro:property name="wheel_length" value="0.06" />
-  <xacro:property name="collision_wheel_length" value="0.145" />
-  <!-- 当たり判定の径 -->
+  <xacro:property name="wheel_width" value="0.06" />
+  <xacro:property name="collision_wheel_width" value="0.145" />
+  <!-- スプロケット径 -->
   <xacro:property name="wheel_radius" value="0.03858" />
-  <!-- スプロケット径 -->
-  <xacro:property name="mini_wheel_radius" value="0.03858" />
   <xacro:property name="wheel_diameter" value="0.07716" />
   <xacro:property name="max_wheel_acceleration" value="1.0" />
   <xacro:property name="max_wheel_torque" value="5.0" />
-  <xacro:property name="big_wheel_front_x" value="0.172" />
-  <xacro:property name="big_wheel_back_x" value="-0.172" />
-  <xacro:property name="center_wheel_z" value="-0.105" />
-  <xacro:property name="big_wheel_z" value="-0.08" />
   <xacro:property name="left_wheel_y" value="0.24" />
   <xacro:property name="right_wheel_y" value="-0.22" />
+  <xacro:property name="front_wheel_x" value="0.172" />
+  <xacro:property name="front_wheel_z" value="-0.08" />
+  <xacro:property name="back_wheel_x" value="-0.172" />
+  <xacro:property name="back_wheel_z" value="-0.08" />
+  <xacro:property name="center_wheel_z" value="-0.105" />
   <link name="base_footprint"/>
   <joint name="base_joint" type="fixed">
@@ -86,11 +85,11 @@
       <origin xyz="0 0 0" rpy="0 0 0"/>
       <geometry>
-        <cylinder length="${wheel_length}" radius="${mini_wheel_radius}"/>
-      </geometry>
-      <material name="dummy_white"/>
-    </visual>
-    <collision>
-      <geometry>
-        <cylinder length="${collision_wheel_length}" radius="${mini_wheel_radius}"/>
+        <cylinder length="${wheel_width}" radius="${wheel_radius}"/>
+      </geometry>
+      <material name="dummy_white"/>
+    </visual>
+    <collision>
+      <geometry>
+        <cylinder length="${collision_wheel_width}" radius="${wheel_radius}"/>
       </geometry>
     </collision>
@@ -105,5 +104,5 @@
     <parent link="base_body"/>
     <child link="left_center_1_wheel"/>
-    <origin xyz="${mini_wheel_radius*2} ${left_wheel_y} ${center_wheel_z}" rpy="0 1.57075 -1.57"/>
+    <origin xyz="${wheel_diameter} ${left_wheel_y} ${center_wheel_z}" rpy="0 1.57075 -1.57"/>
   </joint>
   <link name="left_center_1_wheel">
@@ -111,11 +110,11 @@
       <origin xyz="0 0 0" rpy="0 0 0"/>
       <geometry>
-        <cylinder length="${wheel_length}" radius="${mini_wheel_radius}"/>
-      </geometry>
-      <material name="dummy_white"/>
-    </visual>
-    <collision>
-      <geometry>
-        <cylinder length="${collision_wheel_length}" radius="${mini_wheel_radius}"/>
+        <cylinder length="${wheel_width}" radius="${wheel_radius}"/>
+      </geometry>
+      <material name="dummy_white"/>
+    </visual>
+    <collision>
+      <geometry>
+        <cylinder length="${collision_wheel_width}" radius="${wheel_radius}"/>
       </geometry>
     </collision>
@@ -130,5 +129,5 @@
     <parent link="base_body"/>
     <child link="left_center_3_wheel"/>
-    <origin xyz="-${mini_wheel_radius*2} ${left_wheel_y} ${center_wheel_z}" rpy="0 1.57075 -1.57"/>
+    <origin xyz="-${wheel_diameter} ${left_wheel_y} ${center_wheel_z}" rpy="0 1.57075 -1.57"/>
   </joint>
   <link name="left_center_3_wheel">
@@ -136,11 +135,11 @@
       <origin xyz="0 0 0" rpy="0 0 0"/>
       <geometry>
-        <cylinder length="${wheel_length}" radius="${mini_wheel_radius}"/>
-      </geometry>
-      <material name="dummy_white"/>
-    </visual>
-    <collision>
-      <geometry>
-        <cylinder length="${collision_wheel_length}" radius="${mini_wheel_radius}"/>
+        <cylinder length="${wheel_width}" radius="${wheel_radius}"/>
+      </geometry>
+      <material name="dummy_white"/>
+    </visual>
+    <collision>
+      <geometry>
+        <cylinder length="${collision_wheel_width}" radius="${wheel_radius}"/>
       </geometry>
     </collision>
@@ -155,5 +154,5 @@
     <parent link="base_body"/>
     <child link="left_front_wheel"/>
-    <origin xyz="${big_wheel_front_x} ${left_wheel_y} ${big_wheel_z}" rpy="0 1.57075 -1.57"/>
+    <origin xyz="${front_wheel_x} ${left_wheel_y} ${front_wheel_z}" rpy="0 1.57075 -1.57"/>
   </joint>
   <link name="left_front_wheel">
@@ -161,11 +160,11 @@
       <origin xyz="0 0 0" rpy="0 0 0"/>
       <geometry>
-        <cylinder length="${wheel_length}" radius="${wheel_radius}"/>
-      </geometry>
-      <material name="dummy_white"/>
-    </visual>
-    <collision>
-      <geometry>
-        <cylinder length="${collision_wheel_length}" radius="${wheel_radius}"/>
+        <cylinder length="${wheel_width}" radius="${wheel_radius}"/>
+      </geometry>
+      <material name="dummy_white"/>
+    </visual>
+    <collision>
+      <geometry>
+        <cylinder length="${collision_wheel_width}" radius="${wheel_radius}"/>
       </geometry>
     </collision>
@@ -180,5 +179,5 @@
     <parent link="base_body"/>
     <child link="left_back_wheel"/>
-    <origin xyz="${big_wheel_back_x} ${left_wheel_y} ${big_wheel_z}" rpy="0 1.57075 -1.57"/>
+    <origin xyz="${back_wheel_x} ${left_wheel_y} ${back_wheel_z}" rpy="0 1.57075 -1.57"/>
   </joint>
   <link name="left_back_wheel">
@@ -186,11 +185,11 @@
       <origin xyz="0 0 0" rpy="0 0 0"/>
       <geometry>
-        <cylinder length="${wheel_length}" radius="${wheel_radius}"/>
-      </geometry>
-      <material name="dummy_white"/>
-    </visual>
-    <collision>
-      <geometry>
-        <cylinder length="${collision_wheel_length}" radius="${wheel_radius}"/>
+        <cylinder length="${wheel_width}" radius="${wheel_radius}"/>
+      </geometry>
+      <material name="dummy_white"/>
+    </visual>
+    <collision>
+      <geometry>
+        <cylinder length="${collision_wheel_width}" radius="${wheel_radius}"/>
       </geometry>
     </collision>
@@ -211,11 +210,11 @@
       <origin xyz="0 0 0" rpy="0 0 0"/>
       <geometry>
-        <cylinder length="${wheel_length}" radius="${mini_wheel_radius}"/>
-      </geometry>
-      <material name="dummy_white"/>
-    </visual>
-    <collision>
-      <geometry>
-        <cylinder length="${collision_wheel_length}" radius="${mini_wheel_radius}"/>
+        <cylinder length="${wheel_width}" radius="${wheel_radius}"/>
+      </geometry>
+      <material name="dummy_white"/>
+    </visual>
+    <collision>
+      <geometry>
+        <cylinder length="${collision_wheel_width}" radius="${wheel_radius}"/>
       </geometry>
     </collision>
@@ -230,5 +229,5 @@
     <parent link="base_body"/>
     <child link="right_center_1_wheel"/>
-    <origin xyz="${mini_wheel_radius*2} ${right_wheel_y} ${center_wheel_z}" rpy="0 1.57075 -1.57"/>
+    <origin xyz="${wheel_diameter} ${right_wheel_y} ${center_wheel_z}" rpy="0 1.57075 -1.57"/>
   </joint>
   <link name="right_center_1_wheel">
@@ -236,11 +235,11 @@
       <origin xyz="0 0 0" rpy="0 0 0"/>
       <geometry>
-        <cylinder length="${wheel_length}" radius="${mini_wheel_radius}"/>
-      </geometry>
-      <material name="dummy_white"/>
-    </visual>
-    <collision>
-      <geometry>
-        <cylinder length="${collision_wheel_length}" radius="${mini_wheel_radius}"/>
+        <cylinder length="${wheel_width}" radius="${wheel_radius}"/>
+      </geometry>
+      <material name="dummy_white"/>
+    </visual>
+    <collision>
+      <geometry>
+        <cylinder length="${collision_wheel_width}" radius="${wheel_radius}"/>
       </geometry>
     </collision>
@@ -255,5 +254,5 @@
     <parent link="base_body"/>
     <child link="right_center_3_wheel"/>
-    <origin xyz="-${mini_wheel_radius*2} ${right_wheel_y} ${center_wheel_z}" rpy="0 1.57075 -1.57"/>
+    <origin xyz="-${wheel_diameter} ${right_wheel_y} ${center_wheel_z}" rpy="0 1.57075 -1.57"/>
   </joint>
   <link name="right_center_3_wheel">
@@ -261,11 +260,11 @@
       <origin xyz="0 0 0" rpy="0 0 0"/>
       <geometry>
-        <cylinder length="${wheel_length}" radius="${mini_wheel_radius}"/>
-      </geometry>
-      <material name="dummy_white"/>
-    </visual>
-    <collision>
-      <geometry>
-        <cylinder length="${collision_wheel_length}" radius="${mini_wheel_radius}"/>
+        <cylinder length="${wheel_width}" radius="${wheel_radius}"/>
+      </geometry>
+      <material name="dummy_white"/>
+    </visual>
+    <collision>
+      <geometry>
+        <cylinder length="${collision_wheel_width}" radius="${wheel_radius}"/>
       </geometry>
     </collision>
@@ -280,5 +279,5 @@
     <parent link="base_body"/>
     <child link="right_front_wheel"/>
-    <origin xyz="${big_wheel_front_x} ${right_wheel_y} ${big_wheel_z}" rpy="0 1.57075 -1.57"/>
+    <origin xyz="${front_wheel_x} ${right_wheel_y} ${front_wheel_z}" rpy="0 1.57075 -1.57"/>
   </joint>
   <link name="right_front_wheel">
@@ -286,11 +285,11 @@
       <origin xyz="0 0 0" rpy="0 0 0"/>
       <geometry>
-        <cylinder length="${wheel_length}" radius="${wheel_radius}"/>
-      </geometry>
-      <material name="dummy_white"/>
-    </visual>
-    <collision>
-      <geometry>
-        <cylinder length="${collision_wheel_length}" radius="${wheel_radius}"/>
+        <cylinder length="${wheel_width}" radius="${wheel_radius}"/>
+      </geometry>
+      <material name="dummy_white"/>
+    </visual>
+    <collision>
+      <geometry>
+        <cylinder length="${collision_wheel_width}" radius="${wheel_radius}"/>
       </geometry>
     </collision>
@@ -305,5 +304,5 @@
     <parent link="base_body"/>
     <child link="right_back_wheel"/>
-    <origin xyz="${big_wheel_back_x} ${right_wheel_y} ${big_wheel_z}" rpy="0 1.57075 -1.57"/>
+    <origin xyz="${back_wheel_x} ${right_wheel_y} ${back_wheel_z}" rpy="0 1.57075 -1.57"/>
   </joint>
   <link name="right_back_wheel">
@@ -311,11 +310,11 @@
       <origin xyz="0 0 0" rpy="0 0 0"/>
       <geometry>
-        <cylinder length="${wheel_length}" radius="${wheel_radius}"/>
-      </geometry>
-      <material name="dummy_white"/>
-    </visual>
-    <collision>
-      <geometry>
-        <cylinder length="${collision_wheel_length}" radius="${wheel_radius}"/>
+        <cylinder length="${wheel_width}" radius="${wheel_radius}"/>
+      </geometry>
+      <material name="dummy_white"/>
+    </visual>
+    <collision>
+      <geometry>
+        <cylinder length="${collision_wheel_width}" radius="${wheel_radius}"/>
       </geometry>
     </collision>
